File: hardware/kicad/Sirokko26201_control.kicad_sch (KiCad schematic)
At the start: 21 parts, among them J1 DEVKITC1_J1, J10 MAX31856_EXHAUST_HARNESS, J11 MAX31856_AIR_HARNESS, J12 ROOM_DS18B20_HARNESS, J13 5V_LOGIC_INPUT_ONLY, J20 DRIVER_LOGIC_3V3_ONLY, J21 SAFETY_INTERFACE_3V3_ONLY, J22 PANEL_DRY_CONTACTS_3V3, J3 DEVKITC1_J3

Commit message: hardware: publish DRAFT-02 PCB WIP
Parts:
- added J23: LOCAL_PANEL_ADAFRUIT_938_BUTTONS, TerminalBlock_Phoenix:TerminalBlock_Phoenix_MKDS-1,5-6_1x06_P5.00mm_Horizontal, symbol Connector_Generic:Conn_01x06
- added R13, R14, R15, R16, R17: 10k, Resistor_THT:R_Axial_DIN0207_L6.3mm_D2.5mm_P10.16mm_Horizontal, symbol Device:R
- J1, J3: footprint (none) -> Connector_PinSocket_2.54mm:PinSocket_1x22_P2.54mm_Vertical
- J10, J11, J21: footprint (none) -> TerminalBlock_Phoenix:TerminalBlock_Phoenix_MKDS-1,5-7_1x07_P5.00mm_Horizontal
- J12: footprint (none) -> TerminalBlock_Phoenix:TerminalBlock_Phoenix_MKDS-1,5-3_1x03_P5.00mm_Horizontal
- J13: footprint (none) -> TerminalBlock_Phoenix:TerminalBlock_Phoenix_MKDS-1,5-2_1x02_P5.00mm_Horizontal
- J20: footprint (none) -> TerminalBlock_Phoenix:TerminalBlock_Phoenix_MKDS-1,5-6_1x06_P5.00mm_Horizontal
- J22: footprint (none) -> TerminalBlock_Phoenix:TerminalBlock_Phoenix_MKDS-1,5-4_1x04_P5.00mm_Horizontal
- R1, R10, R11, R12, R2, R3, R4, R5, R6, R7, R8, R9: footprint (none) -> Resistor_THT:R_Axial_DIN0207_L6.3mm_D2.5mm_P10.16mm_Horizontal
Connections:
- net +3V3: now also J23.2 (Pin_2), R13.1, R14.1, R15.1, R16.1, R17.1
- net GND: now also J23.1 (Pin_1)
- net RESET_REQUEST: now also R13.2
- net START_REQUEST: now also R14.2
- net STOP_STATUS: now also R15.2
- net PANEL_SCL: now reaches J3.16 (Pin_16)
- net PANEL_SCL: now also J23.4 (Pin_4)
- net PANEL_SDA: now reaches J3.17 (Pin_17)
- net PANEL_SDA: now also J23.3 (Pin_3)
- net SET_DOWN_REQUEST: now reaches J3.8 (Pin_8)
- net SET_DOWN_REQUEST: now also J23.6 (Pin_6), R17.2
- net SET_UP_REQUEST: now reaches J3.9 (Pin_9)
- net SET_UP_REQUEST: now also J23.5 (Pin_5), R16.2
- no-connect marks 17 -> 13
