File: hardware/kicad/Sirokko26201_control.kicad_sch (KiCad schematic)
At the start: 21 parts, among them J1 DEVKITC1_J1, J10 MAX31856_EXHAUST_HARNESS, J11 MAX31856_AIR_HARNESS, J12 ROOM_DS18B20_HARNESS, J13 5V_LOGIC_INPUT_ONLY, J20 DRIVER_LOGIC_3V3_ONLY, J21 SAFETY_INTERFACE_3V3_ONLY, J22 PANEL_DRY_CONTACTS_3V3, J3 DEVKITC1_J3

Commit message: hardware: preserve recovered main PCB WIP checkpoint
Parts:
- removed J10: MAX31856_EXHAUST_HARNESS, symbol Connector_Generic:Conn_01x07
- removed J11: MAX31856_AIR_HARNESS, symbol Connector_Generic:Conn_01x07
- added C1, C2, C3, C4, C5, C6, C7, C8: 100n 16V X7R, Capacitor_SMD:C_0603_1608Metric, symbol Device:C
- added C10, C15: 0.01uF X7R 16V T+ filter, Capacitor_SMD:C_0603_1608Metric, symbol Device:C
- added C11, C16: 0.01uF X7R 16V T- filter, Capacitor_SMD:C_0603_1608Metric, symbol Device:C
- added C12, C17: 0.1uF X7R 16V AVDD, Capacitor_SMD:C_0603_1608Metric, symbol Device:C
- added C13, C18: 0.1uF X7R 16V DVDD, Capacitor_SMD:C_0603_1608Metric, symbol Device:C
- added C14, C9: 0.1uF X7R 16V BIAS, Capacitor_SMD:C_0603_1608Metric, symbol Device:C
- added J10: TC_K_EXHAUST_T+_T-, TerminalBlock_Phoenix:TerminalBlock_Phoenix_MKDS-1,5-2-5.08_1x02_P5.08mm_Horizontal, symbol Connector_Generic:Conn_01x02
- added J11: TC_K_AIR_T+_T-, TerminalBlock_Phoenix:TerminalBlock_Phoenix_MKDS-1,5-2-5.08_1x02_P5.08mm_Horizontal, symbol Connector_Generic:Conn_01x02
- added J23: LOCAL_BUTTONS_3V3__SET_UP_DOWN_PRESERVED, TerminalBlock_Phoenix:TerminalBlock_Phoenix_MKDS-1,5-6_1x06_P5.00mm_Horizontal, symbol Connector_Generic:Conn_01x06
- added J24: RESET_HW_SPDT_BBM_3V3, TerminalBlock_Phoenix:TerminalBlock_Phoenix_MKDS-1,5-3-5.08_1x03_P5.08mm_Horizontal, symbol Connector_Generic:Conn_01x03
- added J25: THERMAL_AND_HW_ENABLE_3V3_ONLY, TerminalBlock_Phoenix:TerminalBlock_Phoenix_MKDS-1,5-4-5.08_1x04_P5.08mm_Horizontal, symbol Connector_Generic:Conn_01x04
- added J26: TFT_GMT020-02-7P_ST7789V_7P_SOCKET__FOOTPRINT_NOT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, Connector_PinSocket_2.54mm:PinSocket_1x07_P2.54mm_Vertical, symbol Connector_Generic:Conn_01x07
- added R13, R14, R15, R16, R17: 10k, Resistor_THT:R_Axial_DIN0207_L6.3mm_D2.5mm_P10.16mm_Horizontal, symbol Device:R
- added R18, R19, R20, R21, R22: 10k 1%, Resistor_SMD:R_0603_1608Metric, symbol Device:R
- added R23: 33R TFT_RESET_SERIES, Resistor_SMD:R_0603_1608Metric, symbol Device:R
- added R24: 10k TFT_CS_PULLUP, Resistor_SMD:R_0603_1608Metric, symbol Device:R
- added U1: TPS3431SDRBR, Sirokko_Safety:TPS3431_DRB0008A, symbol Sirokko_Safety:TPS3431SDRBR
- added U10, U9: MAX31856MUD+, symbol Sirokko_thermal:MAX31856MUD_PLUS_GRID
- added U2: SN74HCS74D, Package_SO:SOIC-14_3.9x8.7mm_P1.27mm, symbol Sirokko_Safety:SN74HCS74D
- added U3: SN74HCS14D, Package_SO:SOIC-14_3.9x8.7mm_P1.27mm, symbol Sirokko_Safety:SN74HCS14D
- added U4, U5: SN74HCS30D, Package_SO:SOIC-14_3.9x8.7mm_P1.27mm, symbol Sirokko_Safety:SN74HCS30D
- added U6: SN74HCS11D, Package_SO:SOIC-14_3.9x8.7mm_P1.27mm, symbol Sirokko_Safety:SN74HCS11D
- added U7: TPS3839G33DBZR, Package_TO_SOT_SMD:SOT-23, symbol Sirokko_Safety:TPS3839G33DBZR
- added U8: SN74LVC1G14DBVR, Package_TO_SOT_SMD:SOT-23-5, symbol Sirokko_Safety:SN74LVC1G14DBVR
- J1, J3: footprint (none) -> Connector_PinSocket_2.54mm:PinSocket_1x22_P2.54mm_Vertical
- J12: footprint (none) -> TerminalBlock_Phoenix:TerminalBlock_Phoenix_MKDS-1,5-3-5.08_1x03_P5.08mm_Horizontal
- J13: value 5V_LOGIC_INPUT_ONLY -> 24V_LOGIC_INPUT_ONLY__DRAFT_NOT_FOR_ORDER; footprint (none) -> TerminalBlock_Phoenix:TerminalBlock_Phoenix_MKDS-1,5-2-5.08_1x02_P5.08mm_Horizontal
- J20: footprint (none) -> TerminalBlock_Phoenix:TerminalBlock_Phoenix_MKDS-1,5-6_1x06_P5.00mm_Horizontal
- J21: value SAFETY_INTERFACE_3V3_ONLY -> SAFETY_MONITOR_3V3_NO_EXT_DRIVE; footprint (none) -> TerminalBlock_Phoenix:TerminalBlock_Phoenix_MKDS-1,5-7_1x07_P5.00mm_Horizontal
- J22: footprint (none) -> TerminalBlock_Phoenix:TerminalBlock_Phoenix_MKDS-1,5-4-5.08_1x04_P5.08mm_Horizontal
- R1, R10, R11, R12, R2, R3, R4, R5, R6, R7, R8, R9: footprint (none) -> Resistor_THT:R_Axial_DIN0207_L6.3mm_D2.5mm_P10.16mm_Horizontal
Connections:
- net +3V3: now also C1.1, C12.1, C13.1, C17.1, C18.1, C2.1, C3.1, C4.1, C5.1, C6.1, C7.1, C8.1, J23.2 (Pin_2), J25.1 (Pin_1), J26.6 (Pin_6), R13.1, R14.1, R15.1, R16.1, R17.1, R18.1, R19.1, R20.1, R21.1, R24.2, U1.1 (VDD), U1.3 (EN), U1.5 (SET1), U10.5 (AVDD), U10.8 (DVDD), U2.14 (VCC), U2.4 (~{1PRE}), U3.14 (VCC), U4.11 (G), U4.12 (H), U4.14 (VCC), U5.11 (G), U5.12 (H), U5.14 (VCC), U5.6 (F), U6.13 (1C), U6.14 (VCC), U6.5 (2C), U7.3 (VDD), U8.5 (VCC), U9.5 (AVDD), U9.8 (DVDD)
- net ARM_READY: now also U4.5 (E), U5.1 (A)
- net FUEL_CMD: now also U3.3 (2A)
- net FUEL_PERMIT: now also U3.5 (3A), U6.4 (2B)
- net GLOW_CMD: now also U3.9 (4A)
- net GND: now also C1.2, C10.2, C11.2, C12.2, C13.2, C14.2, C15.2, C16.2, C17.2, C18.2, C2.2, C3.2, C4.2, C5.2, C6.2, C7.2, C8.2, C9.2, J23.1 (Pin_1), J24.1 (Pin_1), J25.3 (Pin_3), J26.7 (Pin_7), R22.2, U1.4 (GND), U1.9 (EP), U10.1 (AGND), U10.14 (DGND), U2.11 (2CLK), U2.12 (2D), U2.7 (GND), U3.7 (GND), U4.7 (GND), U5.7 (GND), U6.10 (3B), U6.11 (3C), U6.7 (GND), U6.9 (3A), U7.1 (GND), U8.3 (GND), U9.1 (AGND), U9.14 (DGND)
- net RESET_REQUEST: now also R13.2
- net SAFETY_OK: now also U6.12 (1Y_AND), U6.3 (2A)
- net START_REQUEST: now also R14.2, U5.5 (E)
- net STOP_STATUS: now also R15.2, U8.2 (A)
- net SW_TRIP: now also U3.1 (1A)
- net TC_AIR_CS: now also U10.9 (CS)
- net TC_AIR_DRDY: now also U10.7 (DRDY)
- net TC_EXH_CS: now also U9.9 (CS)
- net TC_EXH_DRDY: now also U9.7 (DRDY)
- net TC_SCK: now also J26.5 (Pin_5), U10.10 (SCK), U9.10 (SCK)
- net TC_SDI_MOSI: now also J26.4 (Pin_4), U10.12 (SDI), U9.12 (SDI)
- net TC_SDO_MISO: now also U10.11 (SDO), U9.11 (SDO)
- net WD_HEARTBEAT: now also U1.6 (WDI)
- net TFT_DC: now reaches J3.16 (Pin_16)
- net TFT_DC: now also J26.2 (Pin_2)
- net TFT_CS: now reaches J3.17 (Pin_17)
- net TFT_CS: now also J26.1 (Pin_1), R24.1
- net SET_DOWN_REQUEST: now reaches J3.8 (Pin_8)
- net SET_DOWN_REQUEST: now also J23.6 (Pin_6), R17.2
- net SET_UP_REQUEST: now reaches J3.9 (Pin_9)
- net SET_UP_REQUEST: now also J23.5 (Pin_5), R16.2
- net EN_CHIP_PU: now reaches J1.3 (Pin_3)
- net EN_CHIP_PU: now also R23.1
- net +5V_LOGIC renamed +5V_DEVKIT
- net +5V_DEVKIT: no longer J13.1 (Pin_1)
- new net ALLOW_LATCH: U2.5 (1Q), U6.1 (1A)
- new net CLEAR_OK: U2.1 (~{1CLR}), U3.10 (5Y), U6.2 (1B)
- new net EXT_SAFETY_ENABLE: J25.4 (Pin_4), U6.6 (2Y_AND)
- new net HW_RESET_CLK: U2.3 (1CLK), U2.9 (2Q)
- new net NOT_CLEAR_OK: U3.11 (5A), U4.8 (Y_NAND)
- new net NOT_FUEL_CMD: U3.4 (2Y), U5.2 (B)
- new net NOT_FUEL_PERMIT: U3.6 (3Y), U5.3 (C)
- new net NOT_GLOW_CMD: U3.8 (4Y), U5.4 (D)
- new net NOT_RESET_ACCEPT: U3.13 (6A), U5.8 (Y_NAND)
- new net NOT_SW_TRIP: U3.2 (1Y), U4.6 (F)
- new net P24_PROTECTED: J13.1 (Pin_1)
- new net PG_OK: U4.1 (A), U7.2 (~{RESET})
- new net RESET_ACCEPT: U2.2 (1D), U3.12 (6Y)
- new net RESET_HW_NC_N: J24.2 (Pin_2), R20.2, U2.13 (~{2CLR})
- new net RESET_HW_NO_N: J24.3 (Pin_3), R21.2, U2.10 (~{2PRE})
- new net STOP_OK: U4.3 (C), U8.4 (Y)
- new net TC_AIR_BIAS: C14.1, U10.2 (BIAS)
- new net TC_AIR_TM: C16.1, J11.2 (Pin_2), U10.3 (T-)
- new net TC_AIR_TP: C15.1, J11.1 (Pin_1), U10.4 (T+)
- new net TC_EXH_BIAS: C9.1, U9.2 (BIAS)
- new net TC_EXH_TM: C11.1, J10.2 (Pin_2), U9.3 (T-)
- new net TC_EXH_TP: C10.1, J10.1 (Pin_1), U9.4 (T+)
- new net TFT_RESET_N: J26.3 (Pin_3), R23.2
- new net THERMAL_OK: J25.2 (Pin_2), R22.1, U4.4 (D)
- new net WD_CWD_FIXED: R18.2, U1.2 (CWD)
- new net WD_OK: R19.2, U1.7 (~{WDO}), U1.8 (ENOUT), U4.2 (B)
- no-connect marks 17 -> 21
Other:
- added sheet LOGIC_POWER_24_TO_5V__DRAFT_NOT_FOR_ORDER (logic_power_24_5_DRAFT.kicad_sch)
- note added: "DRAFT_NOT_FOR_ORDER: LM5013 +5V output is intentionally OPEN at root. No connection to DevKit 5V/VIN until USB reverse-feed arbitration is proven on the exact v1.1 board."
- note added: "HARDWARE FUEL PERMISSION — DRAFT / NO FIRED OPERATION U2.1: fault-dominant allow latch. U2.2: SPDT RESET debounce. RESET: momentary DPDT, break-before-make; hardware pole J24 COM/NC/NO; isolated second pole -> GPIO6 RESET_REQUEST/GND. U7 supervises +3V3 (G33 = 3.08 V nominal); watchdog recovery alone CANNOT re-arm. J21 SAFETY_OK is now a MONITOR OUTPUT. Never drive it externally or bridge to +3V3."
- note added: "J24: 1=GND/COM, 2=NC_N, 3=NO_N. Never short NC_N to NO_N. Both LOW is forbidden for U2.2. J25: 1=+3V3, 2=THERMAL_OK, 3=GND, 4=EXT_SAFETY_ENABLE. 3V3 ONLY — NOT A COIL DRIVER. THERMAL_OK: isolated contact closed to +3V3 when healthy; R22 pulls LOW on open wire. External STOP and independent thermal limit MUST ALSO directly interrupt the protective contactor coil circuit. Output buffering, physical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"
