File: hardware/kicad/MinimalSafety.kicad_sch (KiCad schematic)
At the start: 19 parts, among them U1 TPS3431SDRBR, U11 DRV8803PWPR, U2 SN74HCS74D, U6 SN74HCS11D

Commit message: Remove manual RESET from Sirokko WIP
Parts:
- removed R702: 10k, Resistor_THT:R_Axial_DIN0207_L6.3mm_D2.5mm_P10.16mm_Horizontal, symbol Device:R
Connections:
- net RESET_RELEASED is gone; now on net +3V3: U6.4 (2B)
Other:
- note added: "CLEAR_N = WD_OK & RELAY_DRIVER_OK & P24_PRESENT & MCU_PERMIT"
- note added: "U6.4=+3V3; no manual RESET. ARM_PULSE=GPIO41; MCU_PERMIT=GPIO21; P24_PRESENT=GPIO6 INPUT ONLY."
- note removed: "CLEAR_N = WD_OK & RELAY_DRIVER_OK & RESET_RELEASED & P24_PRESENT & MCU_PERMIT"
- note removed: "Ports: RESET NC -> 3V3; ARM_PULSE=GPIO41; MCU_PERMIT=GPIO21; P24_PRESENT=GPIO6 INPUT ONLY."
