File: hardware/kicad/Sirokko26201_control_motor_candidate.kicad_pcb (KiCad board)
At the start: 2 copper layers, 335 x 170 mm, 144 parts, among them J1 DEVKITC1_J1, J10 TC_K_EXHAUST_T+_T-, J102 MOTOR_24V_HIGH_SPEED; 125W_HE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, J11 TC_K_AIR_T+_T-, J12 ROOM_DS18B20_HARNESS, J13 24V_INPUT_PHOENIX_1756993_WIP, J22 START_STOP B3F-4055 + B32-138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, J23 ENCODER EC11E15244G1 + KNOB 4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, J26 TFT CABLE HARWIN M20-9960845 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, J27 GLOW_OUTPUT_PHOENIX_1756993, J28 CLUTCH_OUTPUT_PHOENIX_1756993, J3 DEVKITC1_J3, K1 DG85BM-5021-76-1024 + DZ85AB-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, K2 DG85BM-5021-76-1024 + DZ85AB-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, K3 DG85BM-5021-76-1024 + DZ85AB-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, Q1 IPB017N10N5LFATMA1 WIP, Q101 IRFB4110PBF (100V; RDS(on) @ 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, Q2 IPB017N10N5LFATMA1 WIP, Q20 BC847B,215, Q3 IPB017N10N5LFATMA1 WIP, Q4 IPB017N10N5LFATMA1 WIP, U10 MAX31856MUD+, U101 LM5013DDAR, U11 DRV8803PWPR, U13 LM74800QDRRRQ1 WIP_NOT_TRANSI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, U20 SN74LVC1G97DBVR, U301 TPS62162DSGR, U302 TPS3808G33DBVR, U303 74LVC125APW,118 Nexperia ONLY, U9 MAX31856MUD+, U9001 LTC7001IMSE#PBF; MSOP-10 EP, U9002 INA240A1ID, U9003 TLV9020DBVR, U9004 SN74LVC1G32DBVR, U9005 SN74LVC1G08DBVR, U9006 SN74LVC1G08DBVR, U9007 LM317HVT/NOPB TO-220; TJ 0…12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

Commit message: Publish GND PCB WIP snapshot
Routing:
- net /GND: track 2085.9 -> 2170.3 mm, vias 70 -> 75
Changed lines of the file:
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@@
 		(net "/+3V3")
 	)
+	(segment
+		(start 76.5 35)
+		(end 76.5 35.5)
+		(width 0.4)
+		(layer "B.Cu")
+		(net "/GND")
+	)
+	(segment
+		(start 76 13.5)
+		(end 77 13.5)
+		(width 0.6)
+		(layer "F.Cu")
+		(net "/GND")
+	)
+	(segment
+		(start 77 13.5)
+		(end 79 11.55)
+		(width 0.6)
+		(layer "F.Cu")
+		(net "/GND")
+	)
+	(via
+		(at 105.86 91)
+		(size 0.6)
+		(drill 0.3)
+		(layers "F.Cu" "B.Cu")
+		(net "/GND")
+	)
+	(segment
+		(start 105.86 91)
+		(end 107.34 91)
+		(width 0.6)
+		(layer "F.Cu")
+		(net "/GND")
+	)
+	(segment
+		(start 107.34 91)
+		(end 110 88.34)
+		(width 0.6)
+		(layer "F.Cu")
+		(net "/GND")
+	)
+	(via
+		(at 110 88.34)
+		(size 0.6)
+		(drill 0.3)
+		(layers "F.Cu" "B.Cu")
+		(net "/GND")
+	)
+	(segment
+		(start 53.16 80)
+		(end 53.36 79.8)
+		(width 0.4)
+		(layer "F.Cu")
+		(net "/GND")
+	)
+	(segment
+		(start 53.36 79.8)
+		(end 71 79.8)
+		(width 0.4)
+		(layer "F.Cu")
+		(net "/GND")
+	)
+	(via
+		(at 61.7 79.8)
+		(size 0.6)
+		(drill 0.3)
+		(layers "F.Cu" "B.Cu")
+		(net "/GND")
+	)
+	(segment
+		(start 36.775 91.05)
+		(end 35.8 90.075)
+		(width 0.3)
+		(layer "F.Cu")
+		(net "/GND")
+	)
+	(segment
+		(start 35.8 90.075)
+		(end 35.8 79.8)
+		(width 0.3)
+		(layer "F.Cu")
+		(net "/GND")
+	)
+	(segment
+		(start 35.8 79.8)
+		(end 40.5 79.8)
+		(width 0.3)
+		(layer "F.Cu")
+		(net "/GND")
+	)
+	(segment
+		(start 34.4 113.6)
+		(end 34.4 104.8)
+		(width 0.4)
+		(layer "F.Cu")
+		(net "/GND")
+	)
+	(via
+		(at 34.4 104.8)
+		(size 0.6)
+		(drill 0.3)
+		(layers "F.Cu" "B.Cu")
+		(net "/GND")
+	)
+	(segment
+		(start 34.4 104.8)
+		(end 36 104.8)
+		(width 0.4)
+		(layer "B.Cu")
+		(net "/GND")
+	)
+	(segment
+		(start 67.45 103)
+		(end 67.45 113.7)
+		(width 0.4)
+		(layer "F.Cu")
+		(net "/GND")
+	)
+	(via
+		(at 67.45 113.7)
+		(size 0.6)
+		(drill 0.3)
+		(layers "F.Cu" "B.Cu")
+		(net "/GND")
+	)
+	(segment
+		(start 177.6 138.05)
+		(end 175.7 138.05)
+		(width 0.25)
+		(layer "B.Cu")
+		(net "/GND")
+	)
+	(segment
+		(start 175.7 138.05)
+		(end 175.7 141.95)
+		(width 0.25)
+		(layer "B.Cu")
+		(net "/GND")
+	)
+	(segment
+		(start 175.7 141.95)
+		(end 177.6 141.95)
+		(width 0.25)
+		(layer "B.Cu")
+		(net "/GND")
+	)
+	(segment
+		(start 175.7 140)
+		(end 177.6 140)
+		(width 0.25)
+		(layer "B.Cu")
+		(net "/GND")
+	)
+	(segment
+		(start 186 157.5)
+		(end 186 154.6)
+		(width 0.3)
+		(layer "F.Cu")
+		(net "/GND")
+	)
+	(segment
+		(start 186 154.6)
+		(end 182.4 151)
+		(width 0.3)
+		(layer "F.Cu")
+		(net "/GND")
+	)
+	(segment
+		(start 182.4 151)
+		(end 180.5 151)
+		(width 0.3)
+		(layer "F.Cu")
+		(net "/GND")
+	)
 )

Commit message: hardware: publish 1527 GND WIP
Routing:
- net /GND: track 2170.3 -> 2199.9 mm
Changed lines of the file:
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@@
+		(net "/GND")
+	)
+	(segment
+		(start 267.525 29.9)
+		(end 263 25.375)
+		(width 0.4)
+		(layer "B.Cu")
+		(net "/GND")
+	)
+	(segment
+		(start 263 25.375)
+		(end 263 21.5)
+		(width 0.4)
+		(layer "B.Cu")
+		(net "/GND")
+	)
+	(segment
+		(start 76 27.45)
+		(end 76.3 27.15)
+		(width 0.4)
+		(layer "B.Cu")
+		(net "/GND")
+	)
+	(segment
+		(start 76.3 27.15)
+		(end 76.3 20.44)
+		(width 0.4)
+		(layer "B.Cu")
+		(net "/GND")
+	)
+	(segment
+		(start 76.3 20.44)
+		(end 81.55 20.44)
+		(width 0.4)
+		(layer "B.Cu")
+		(net "/GND")
+	)
+	(segment
+		(start 81.55 20.44)
+		(end 81.55 27.45)
+		(width 0.4)
+		(layer "B.Cu")
 		(net "/GND")
 	)

Commit message: hardware: publish 1531 +3V3 WIP
Routing:
- net /+3V3: track 1188.7 -> 1217.9 mm
Changed lines of the file:
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@@
 		(net "/GND")
 	)
+	(segment
+		(start 76 13.5)
+		(end 76.68 12.82)
+		(width 0.4)
+		(layer "B.Cu")
+		(net "/+3V3")
+	)
+	(segment
+		(start 76.68 12.82)
+		(end 102 12.82)
+		(width 0.4)
+		(layer "B.Cu")
+		(net "/+3V3")
+	)
+	(segment
+		(start 102 12.82)
+		(end 103.27 14.09)
+		(width 0.4)
+		(layer "B.Cu")
+		(net "/+3V3")
+	)
+	(segment
+		(start 103.27 14.09)
+		(end 104.4 14.09)
+		(width 0.4)
+		(layer "B.Cu")
+		(net "/+3V3")
+	)
 )

Commit message: hardware: publish 1537 GND bridge WIP
Routing:
- net /GND: track 2199.9 -> 2240.8 mm
Changed lines of the file:
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@@
 		(net "/+3V3")
 	)
+	(segment
+		(start 251 36)
+		(end 254.5 36)
+		(width 0.5)
+		(layer "F.Cu")
+		(net "/GND")
+	)
+	(segment
+		(start 254.5 36)
+		(end 254.5 30)
+		(width 0.5)
+		(layer "F.Cu")
+		(net "/GND")
+	)
+	(segment
+		(start 254.5 30)
+		(end 252.5 28)
+		(width 0.5)
+		(layer "F.Cu")
+		(net "/GND")
+	)
+	(segment
+		(start 252.5 28)
+		(end 249.875 27.275)
+		(width 0.5)
+		(layer "F.Cu")
+		(net "/GND")
+	)
+	(segment
+		(start 104.4 64.89)
+		(end 104.4 82.74)
+		(width 0.5)
+		(layer "F.Cu")
+		(net "/GND")
+	)
+	(segment
+		(start 104.4 82.74)
+		(end 110 88.34)
+		(width 0.5)
+		(layer "F.Cu")
+		(net "/GND")
+	)
 )

Commit message: hardware: publish 1536 orphan-track cleanup WIP
Routing:
- net /+3V3: track 1217.9 -> 1216.9 mm
Changed lines of the file:
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@@
-	)
-	(segment
-		(start 286.1375 24.05)
-		(end 287.2 24.05)
-		(width 0.25)
-		(layer "F.Cu")
-		(net "/+3V3")
 	)
 	(segment

Commit message: hardware: remove external EN_CHIP_PU path
Connections:
- J1 pad 3: /EN_CHIP_PU -> unconnected-(J1-Pin_3-Pad3)
Routing:
- net /EN_CHIP_PU: track 182.4 -> 0.00 mm, vias 5 -> 0

Commit message: Move R9004 beside Q101
Parts:
- moved R9004 9.34 mm to (252.5, 145.0)
Routing:
- net /MOTOR_PWM_REBUILD_CANDIDATE/TGUP: track 17.1 -> 8.88 mm, vias 2 -> 0
- net /MOTOR_PWM_REBUILD_CANDIDATE/GATE_Q101: track 26.9 -> 21.8 mm
Changed lines of the file:
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@@
 	(footprint "Resistor_SMD:R_0603_1608Metric"
 		(layer "F.Cu")
-		(at 250 154)
+		(at 252.5 145)
 		(descr "Resistor SMD 0603 (1608 Metric), square (rectangular) end terminal, IPC-7351 nominal, (Body size source: IPC-SM-782 page 72, https://www.pcb-3d.com/wordpress/wp-content/uploads/ipc-sm-782a_amendment_1_and_2.pdf)")
 		(tags "resistor")
@@
 	)
 	(segment
-		(start 248.8 154)
-		(end 249.175 154)
+		(start 249 142.2)
+		(end 249 142.325)
 		(width 0.2)
 		(layer "F.Cu")
@@
 	)
 	(segment
-		(start 248.8 152.8)
-		(end 248.8 154)
+		(start 247.5 140.7)
+		(end 249 142.2)
 		(width 0.2)
 		(layer "F.Cu")
@@
 	)
 	(segment
-		(start 245.15 139.5)
-		(end 246.3 139.5)
+		(start 249 142.325)
+		(end 251.675 145)
 		(width 0.2)
 		(layer "F.Cu")
 		(net "/MOTOR_PWM_REBUILD_CANDIDATE/TGUP")
 	)
-	(via
-		(at 248.8 152.8)
-		(size 0.6)
-		(drill 0.3)
-		(layers "F.Cu" "B.Cu")
-		(net "/MOTOR_PWM_REBUILD_CANDIDATE/TGUP")
-	)
-	(via
-		(at 247.5 140.7)
-		(size 0.6)
-		(drill 0.3)
-		(layers "F.Cu" "B.Cu")
-		(net "/MOTOR_PWM_REBUILD_CANDIDATE/TGUP")
-	)
 	(segment
-		(start 247.5 140.7)
-		(end 248.8 142)
-		(width 0.2)
-		(layer "B.Cu")
-		(net "/MOTOR_PWM_REBUILD_CANDIDATE/TGUP")
-	)
-	(segment
-		(start 248.8 142)
-		(end 248.8 152.8)
+		(start 245.15 139.5)
+		(end 246.3 139.5)
 		(width 0.2)
-		(layer "B.Cu")
+		(layer "F.Cu")
 		(net "/MOTOR_PWM_REBUILD_CANDIDATE/TGUP")
 	)
@@
 	)
 	(segment
-		(start 253 145)
-		(end 257 145)
-		(width 0.4)
+		(start 247.8 146.7)
+		(end 255.3 146.7)
+		(width 0.2)
 		(layer "F.Cu")
 		(net "/MOTOR_PWM_REBUILD_CANDIDATE/GATE_Q101")
 	)
 	(segment
-		(start 247.8 143)
-		(end 253 143)
+		(start 255.3 146.7)
+		(end 257 145)
 		(width 0.2)
 		(layer "F.Cu")
@@
 	)
 	(segment
-		(start 250.825 154)
-		(end 253 154)
-		(width 0.4)
-		(layer "F.Cu")
-		(net "/MOTOR_PWM_REBUILD_CANDIDATE/GATE_Q101")
-	)
-	(segment
-		(start 253 143)
-		(end 253 145)
+		(start 247.8 143)
+		(end 247.8 146.7)
 		(width 0.2)
 		(layer "F.Cu")
@@
 	)
 	(segment
-		(start 253 154)
-		(end 253 145)
+		(start 253.325 145)
+		(end 257 145)
 		(width 0.4)
 		(layer "F.Cu")
