File: hardware/kicad/Sirokko26201_control_motor_candidate.kicad_sch (KiCad schematic)
At the start: 49 parts, among them J1 DEVKITC1_J1, J10 TC_K_EXHAUST_T+_T-, J11 TC_K_AIR_T+_T-, J12 ROOM_DS18B20_HARNESS, J13 24V_INPUT_PHOENIX_1756993_WIP, J22 START_STOP B3F-4055 + B32-138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, J23 ENCODER EC11E15244G1 + KNOB 4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, J24 RESET NKK BB25AB-FA, J26 TFT CABLE HARWIN M20-9960845 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, J27 GLOW_OUTPUT_PHOENIX_1756993, J28 CLUTCH_OUTPUT_PHOENIX_1756993, J3 DEVKITC1_J3, K1 DG85BM-5021-76-1024 + DZ85AB-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, K2 DG85BM-5021-76-1024 + DZ85AB-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, K3 DG85BM-5021-76-1024 + DZ85AB-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, Q20 BC847B,215, U10 MAX31856MUD+, U20 SN74LVC1G97DBVR, U9 MAX31856MUD+

Commit message: Remove manual RESET from Sirokko WIP
Parts:
- removed J24: RESET NKK BB25AB-FA, Sirokko_Panel:SW_NKK_BB25AB-FA_3D_ENVELOPE, symbol Switch:SW_Push_DPDT
Connections:
- no-connect marks 22 -> 20
Other:
- sheet MinimalSafety ports: added none; removed RESET_RELEASED
- note added: "Manual RESET removed: no J24, external reset header, jumper or replacement button. Automatic safety remains: watchdog, latch and CLEAR_N conditions are preserved. U6.4 is fixed HIGH by +3V3; valid arming requires a new ARM_PULSE from ESP32. EN_CHIP_PU remains at J1.3 for DevKit/USB service; firmware synchronization is pending."
- note removed: "J24 RESET ACTUAL PIN CONTRACT (NKK BB25AB-FA) 1=EN_CHIP_PU NO; 2=GND COM; 3=unused NC. Hardware RESET grounds DevKit EN. 4=unused NO; 5=3V3 COM; 6=RESET_RELEASED NC, pulled LOW by R702 when open. J25 REMOVED: no external power or permit interface. Temperature conditions belong to MCU_PERMIT, asserted only by the qualified control cycle. U6.1 and U6.2 both receive WD_OK; no permanently asserted ne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"
Changed lines of the file:
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@@
 )
 (symbol
-	(lib_name "Switch:SW_Push_DPDT")
-	(lib_id "Switch:SW_Push_DPDT")
-	(at 530.86 129.54 0)
-	(unit 1)
-	(exclude_from_sim no)
-	(in_bom yes)
-	(on_board yes)
-	(dnp no)
-	(property "Reference" "J24"
-		(at 530.86 125.73 0)
-		(effects
-			(font
-				(size 1.27 1.27)
-			)
-		)
-	)
-	(property "Value" "RESET NKK BB25AB-FA"
-		(at 530.86 133.35 0)
-		(effects
-			(font
-				(size 1.27 1.27)
-			)
-		)
-	)
-	(property "Footprint" "Sirokko_Panel:SW_NKK_BB25AB-FA_3D_ENVELOPE"
-		(at 530.86 129.54 0)
-		(effects
-			(font
-				(size 1.27 1.27)
-			)
-			(hide yes)
-		)
-	)
-	(property "Datasheet" "~"
-		(at 530.86 129.54 0)
-		(effects
-			(font
-				(size 1.27 1.27)
-			)
-			(hide yes)
-		)
-	)
-	(property "MPN" "BB25AB-FA"
-	(id 0)
-	(at 530.86 129.54 0)
-	(effects
-		(font
-			(size 1.27 1.27)
-		)
-		(hide yes)
-	)
-)
-	(pin "1"
-)
-	(pin "2"
-)
-	(pin "3"
-)
-	(pin "4"
-)
-	(pin "5"
-)
-	(pin "6"
-)
-	(instances
-		(project "Sirokko26201_control_motor_candidate"
-			(path "/d7270d3f-3491-4796-ae0a-c336632ea3f7"
-				(reference "J24")
-				(unit 1)
-			)
-		)
-	)
-)
-(symbol
 	(lib_name "Device:R")
 	(lib_id "Device:R")
@@
 			(footprint "Sirokko_Panel:RotaryEncoder_Alps_EC11E15244G1_Knob41001_3D_ENVELOPE")
 		)
-		(path "/d7270d3f-3491-4796-ae0a-c336632ea3f7/683915be-cf9f-491a-8cd4-61f74f9bb932"
-			(reference "J24")
-			(unit 1)
-			(value "RESET NKK BB25AB-FA")
-			(footprint "Sirokko_Panel:SW_NKK_BB25AB-FA_3D_ENVELOPE")
-		)
 		(path "/d7270d3f-3491-4796-ae0a-c336632ea3f7/99b8e38a-90e8-455c-bbb6-cf829b4f14a0"
 			(reference "R85")
@@
 (wire
 	(pts
-		(xy 525.78 124.46) (xy 523.24 124.46)
-	)
-	(stroke
-		(width 0)
-		(type default)
-	)
-)
-(wire
-	(pts
 		(xy 558.8 100.33) (xy 558.8 102.87)
 	)
@@
 (wire
 	(pts
-		(xy 535.94 137.16) (xy 538.48 137.16)
-	)
-	(stroke
-		(width 0)
-		(type default)
-	)
-)
-(wire
-	(pts
 		(xy 430.53 64.77) (xy 427.99 64.77)
 	)
@@
 	)
 (label "GND"
-		(at 523.24 124.46 180)
-		(effects
-			(font
-				(size 1.27 1.27)
-			)
-			(justify right bottom)
-		)
-	)
-(label "GND"
 		(at 558.8 102.87 270)
 		(effects
@@
 		)
 	)
-(label "RESET_RELEASED"
-		(at 538.48 137.16 0)
-		(effects
-			(font
-				(size 1.27 1.27)
-			)
-			(justify left bottom)
-		)
-	)
 (label "GND"
 		(at 394.97 402.59 0)
@@
 )
 (no_connect
-	(at 535.94 127)
-)
-(no_connect
 	(at 377.19 139.7)
 )
@@
 	 (justify left top))
 )
-(text "J24 RESET ACTUAL PIN CONTRACT (NKK BB25AB-FA)\n1=EN_CHIP_PU NO; 2=GND COM; 3=unused NC. Hardware RESET grounds DevKit EN.\n4=unused NO; 5=3V3 COM; 6=RESET_RELEASED NC, pulled LOW by R702 when open.\nJ25 REMOVED: no external power or permit interface.\nTemperature conditions belong to MCU_PERMIT, asserted only by the qualified control cycle.\nU6.1 and U6.2 both receive WD_OK; no permanently asserted new input. R701 removed. Reset timing is unqualified."
-	(at 25.4 375.92 0)
-	(effects
-		(font
-			(size 1.27 1.27)
-		)
-	 (justify left top))
-)
 (text "DRAFT: LM5013 5V is assigned to +5V_DEVKIT in this hierarchy. USB reverse-feed arbitration remains UNQUALIFIED. NO POWER."
 	(at 430 35 0)
@@
 	 (justify left top))
 )
+(text "Manual RESET removed: no J24, external reset header, jumper or replacement button.\nAutomatic safety remains: watchdog, latch and CLEAR_N conditions are preserved.\nU6.4 is fixed HIGH by +3V3; valid arming requires a new ARM_PULSE from ESP32.\nEN_CHIP_PU remains at J1.3 for DevKit/USB service; firmware synchronization is pending."
+	(at 25.4 375.92 0)
+	(effects
+		(font
+			(size 1.27 1.27)
+		)
+	)
+)
 (junction
 	(at 114.46 59.69)
@@
 (embedded_fonts no)
 (no_connect (at 251.46 76.2))
-(no_connect (at 535.94 132.08))
-(wire (pts (xy 525.78 134.62) (xy 520.7 134.62)) (stroke (width 0) (type default)))
-(label "+3V3" (at 520.7 134.62 0) (effects (font (size 1 1)) (justify right bottom)))
 (wire (pts (xy 195.58 279.4) (xy 190.5 279.4)) (stroke (width 0) (type default)))
 (label "+3V3" (at 190.5 279.4 0) (effects (font (size 1 1)) (justify right bottom)))
@@
 (wire (pts (xy 195.58 309.88) (xy 190.5 309.88)) (stroke (width 0) (type default)))
 (label "WD_HEARTBEAT" (at 190.5 309.88 0) (effects (font (size 1 1)) (justify right bottom)))
-(wire (pts (xy 195.58 325.12) (xy 190.5 325.12)) (stroke (width 0) (type default)))
-(label "RESET_RELEASED" (at 190.5 325.12 0) (effects (font (size 1 1)) (justify right bottom)))
 (wire (pts (xy 195.58 332.74) (xy 190.5 332.74)) (stroke (width 0) (type default)))
 (label "MCU_PERMIT" (at 190.5 332.74 0) (effects (font (size 1 1)) (justify right bottom)))
@@
 (wire (pts (xy 381.0 302.26) (xy 386.08 302.26)) (stroke (width 0) (type default)))
 (label "K_CLUTCH_SAFE_COIL_LOW" (at 386.08 302.26 0) (effects (font (size 1 1)) (justify left bottom)))
-(sheet (at 195.58 271.78) (size 185.42 91.44) (stroke (width 0.1524) (type solid)) (fill (color 0 0 0 0)) (property "Sheetname" "MinimalSafety" (at 195.58 270.51 0) (effects (font (size 1.27 1.27)) (justify left bottom))) (property "Sheetfile" "MinimalSafety.kicad_sch" (at 195.58 364.49 0) (effects (font (size 1 1)) (justify left top))) (pin "+3V3" input (at 195.58 279.4 180) (effects (font (size 1 1)) (justify left))) (pin "GND" input (at 195.58 287.02 180) (effects (font (size 1 1)) (justify left))) (pin "P24_PROTECTED" input (at 195.58 294.64 180) (effects (font (size 1 1)) (justify left))) (pin "P24_PRESENT" input (at 195.58 302.26 180) (effects (font (size 1 1)) (justify left))) (pin "WD_HEARTBEAT" input (at 195.58 309.88 180) (effects (font (size 1 1)) (justify left)))  (pin "RESET_RELEASED" input (at 195.58 325.12 180) (effects (font (size 1 1)) (justify left))) (pin "MCU_PERMIT" input (at 195.58 332.74 180) (effects (font (size 1 1)) (justify left))) (pin "ARM_PULSE" input (at 195.58 340.36 180) (effects (font (size 1 1)) (justify left))) (pin "GLOW_CMD" input (at 195.58 347.98 180) (effects (font (size 1 1)) (justify left))) (pin "FUEL_CMD" input (at 195.58 355.6 180) (effects (font (size 1 1)) (justify left))) (pin "SAFETY_OK" output (at 381.0 279.4 0) (effects (font (size 1 1)) (justify right))) (pin "K_GLOW_COIL_LOW" output (at 381.0 287.02 0) (effects (font (size 1 1)) (justify right))) (pin "K_CLUTCH_RUN_COIL_LOW" output (at 381.0 294.64 0) (effects (font (size 1 1)) (justify right))) (pin "K_CLUTCH_SAFE_COIL_LOW" output (at 381.0 302.26 0) (effects (font (size 1 1)) (justify right))))
+(sheet (at 195.58 271.78) (size 185.42 91.44) (stroke (width 0.1524) (type solid)) (fill (color 0 0 0 0)) (property "Sheetname" "MinimalSafety" (at 195.58 270.51 0) (effects (font (size 1.27 1.27)) (justify left bottom))) (property "Sheetfile" "MinimalSafety.kicad_sch" (at 195.58 364.49 0) (effects (font (size 1 1)) (justify left top))) (pin "+3V3" input (at 195.58 279.4 180) (effects (font (size 1 1)) (justify left))) (pin "GND" input (at 195.58 287.02 180) (effects (font (size 1 1)) (justify left))) (pin "P24_PROTECTED" input (at 195.58 294.64 180) (effects (font (size 1 1)) (justify left))) (pin "P24_PRESENT" input (at 195.58 302.26 180) (effects (font (size 1 1)) (justify left))) (pin "WD_HEARTBEAT" input (at 195.58 309.88 180) (effects (font (size 1 1)) (justify left))) (pin "MCU_PERMIT" input (at 195.58 332.74 180) (effects (font (size 1 1)) (justify left))) (pin "ARM_PULSE" input (at 195.58 340.36 180) (effects (font (size 1 1)) (justify left))) (pin "GLOW_CMD" input (at 195.58 347.98 180) (effects (font (size 1 1)) (justify left))) (pin "FUEL_CMD" input (at 195.58 355.6 180) (effects (font (size 1 1)) (justify left))) (pin "SAFETY_OK" output (at 381.0 279.4 0) (effects (font (size 1 1)) (justify right))) (pin "K_GLOW_COIL_LOW" output (at 381.0 287.02 0) (effects (font (size 1 1)) (justify right))) (pin "K_CLUTCH_RUN_COIL_LOW" output (at 381.0 294.64 0) (effects (font (size 1 1)) (justify right))) (pin "K_CLUTCH_SAFE_COIL_LOW" output (at 381.0 302.26 0) (effects (font (size 1 1)) (justify right))))
 (wire (pts (xy 180.34 76.2) (xy 175.26 76.2)) (stroke (width 0) (type default)))
 (label "P24_PRESENT" (at 175.26 76.2 0) (effects (font (size 1 1)) (justify right bottom)))
 (no_connect (at 251.46 101.6))
-(wire (pts (xy 535.94 121.92) (xy 541.02 121.92)) (stroke (width 0) (type default)))
-(label "EN_CHIP_PU" (at 541.02 121.92 0) (effects (font (size 1 1)) (justify left bottom)))
 )

Commit message: WIP: publish current unfinished CAD sources
Connections:
- net ARM_PULSE: no longer names the net of J3.7 (Pin_7)
- net SAFETY_OK: no longer names the net of J1.5 (Pin_5)
- net WD_HEARTBEAT: no longer names the net of J1.11 (Pin_11)
- no-connect marks 20 -> 23
Other:
- sheet MinimalSafety ports: added none; removed +3V3, ARM_PULSE, P24_PRESENT, SAFETY_OK, WD_HEARTBEAT
Changed lines of the file:
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@@
 (wire
 	(pts
-		(xy 180.34 73.66) (xy 175.26 73.66)
-	)
-	(stroke
-		(width 0)
-		(type default)
-	)
-)
-(wire
-	(pts
 		(xy 180.34 78.74) (xy 175.26 78.74)
 	)
@@
 (wire
 	(pts
-		(xy 180.34 88.9) (xy 175.26 88.9)
-	)
-	(stroke
-		(width 0)
-		(type default)
-	)
-)
-(wire
-	(pts
-		(xy 251.46 78.74) (xy 246.38 78.74)
-	)
-	(stroke
-		(width 0)
-		(type default)
-	)
-)
-(wire
-	(pts
 		(xy 60.96 245.11) (xy 60.96 242.57)
 	)
@@
 	)
 )
-(label "SAFETY_OK"
-	(at 175.26 73.66 180)
-	(effects
-		(font
-			(size 1.27 1.27)
-		)
-	)
-)
 (label "START_REQUEST"
 	(at 175.26 78.74 180)
@@
 	)
 )
-(label "WD_HEARTBEAT"
-	(at 175.26 88.9 180)
-	(effects
-		(font
-			(size 1.27 1.27)
-		)
-	)
-)
-(label "ARM_PULSE"
-	(at 246.38 78.74 180)
-	(effects
-		(font
-			(size 1.27 1.27)
-		)
-	)
-)
 (label "+3V3"
 	(at 60.96 242.57 90)
@@
 (embedded_fonts no)
 (no_connect (at 251.46 76.2))
-(wire (pts (xy 195.58 279.4) (xy 190.5 279.4)) (stroke (width 0) (type default)))
-(label "+3V3" (at 190.5 279.4 0) (effects (font (size 1 1)) (justify right bottom)))
 (wire (pts (xy 195.58 287.02) (xy 190.5 287.02)) (stroke (width 0) (type default)))
 (label "GND" (at 190.5 287.02 0) (effects (font (size 1 1)) (justify right bottom)))
 (wire (pts (xy 195.58 294.64) (xy 190.5 294.64)) (stroke (width 0) (type default)))
 (label "P24_PROTECTED" (at 190.5 294.64 0) (effects (font (size 1 1)) (justify right bottom)))
-(wire (pts (xy 195.58 302.26) (xy 190.5 302.26)) (stroke (width 0) (type default)))
-(label "P24_PRESENT" (at 190.5 302.26 0) (effects (font (size 1 1)) (justify right bottom)))
-(wire (pts (xy 195.58 309.88) (xy 190.5 309.88)) (stroke (width 0) (type default)))
-(label "WD_HEARTBEAT" (at 190.5 309.88 0) (effects (font (size 1 1)) (justify right bottom)))
 (wire (pts (xy 195.58 332.74) (xy 190.5 332.74)) (stroke (width 0) (type default)))
 (label "MCU_PERMIT" (at 190.5 332.74 0) (effects (font (size 1 1)) (justify right bottom)))
-(wire (pts (xy 195.58 340.36) (xy 190.5 340.36)) (stroke (width 0) (type default)))
-(label "ARM_PULSE" (at 190.5 340.36 0) (effects (font (size 1 1)) (justify right bottom)))
 (wire (pts (xy 195.58 347.98) (xy 190.5 347.98)) (stroke (width 0) (type default)))
 (label "GLOW_CMD" (at 190.5 347.98 0) (effects (font (size 1 1)) (justify right bottom)))
 (wire (pts (xy 195.58 355.6) (xy 190.5 355.6)) (stroke (width 0) (type default)))
 (label "FUEL_CMD" (at 190.5 355.6 0) (effects (font (size 1 1)) (justify right bottom)))
-(wire (pts (xy 381.0 279.4) (xy 386.08 279.4)) (stroke (width 0) (type default)))
-(label "SAFETY_OK" (at 386.08 279.4 0) (effects (font (size 1 1)) (justify left bottom)))
 (wire (pts (xy 381.0 287.02) (xy 386.08 287.02)) (stroke (width 0) (type default)))
 (label "K_GLOW_COIL_LOW" (at 386.08 287.02 0) (effects (font (size 1 1)) (justify left bottom)))
@@
 (wire (pts (xy 381.0 302.26) (xy 386.08 302.26)) (stroke (width 0) (type default)))
 (label "K_CLUTCH_SAFE_COIL_LOW" (at 386.08 302.26 0) (effects (font (size 1 1)) (justify left bottom)))
-(sheet (at 195.58 271.78) (size 185.42 91.44) (stroke (width 0.1524) (type solid)) (fill (color 0 0 0 0)) (property "Sheetname" "MinimalSafety" (at 195.58 270.51 0) (effects (font (size 1.27 1.27)) (justify left bottom))) (property "Sheetfile" "MinimalSafety.kicad_sch" (at 195.58 364.49 0) (effects (font (size 1 1)) (justify left top))) (pin "+3V3" input (at 195.58 279.4 180) (effects (font (size 1 1)) (justify left))) (pin "GND" input (at 195.58 287.02 180) (effects (font (size 1 1)) (justify left))) (pin "P24_PROTECTED" input (at 195.58 294.64 180) (effects (font (size 1 1)) (justify left))) (pin "P24_PRESENT" input (at 195.58 302.26 180) (effects (font (size 1 1)) (justify left))) (pin "WD_HEARTBEAT" input (at 195.58 309.88 180) (effects (font (size 1 1)) (justify left))) (pin "MCU_PERMIT" input (at 195.58 332.74 180) (effects (font (size 1 1)) (justify left))) (pin "ARM_PULSE" input (at 195.58 340.36 180) (effects (font (size 1 1)) (justify left))) (pin "GLOW_CMD" input (at 195.58 347.98 180) (effects (font (size 1 1)) (justify left))) (pin "FUEL_CMD" input (at 195.58 355.6 180) (effects (font (size 1 1)) (justify left))) (pin "SAFETY_OK" output (at 381.0 279.4 0) (effects (font (size 1 1)) (justify right))) (pin "K_GLOW_COIL_LOW" output (at 381.0 287.02 0) (effects (font (size 1 1)) (justify right))) (pin "K_CLUTCH_RUN_COIL_LOW" output (at 381.0 294.64 0) (effects (font (size 1 1)) (justify right))) (pin "K_CLUTCH_SAFE_COIL_LOW" output (at 381.0 302.26 0) (effects (font (size 1 1)) (justify right))))
+(sheet (at 195.58 271.78) (size 185.42 91.44) (stroke (width 0.1524) (type solid)) (fill (color 0 0 0 0)) (property "Sheetname" "MinimalSafety" (at 195.58 270.51 0) (effects (font (size 1.27 1.27)) (justify left bottom))) (property "Sheetfile" "MinimalSafety.kicad_sch" (at 195.58 364.49 0) (effects (font (size 1 1)) (justify left top))) (pin "GND" input (at 195.58 287.02 180) (effects (font (size 1 1)) (justify left))) (pin "P24_PROTECTED" input (at 195.58 294.64 180) (effects (font (size 1 1)) (justify left))) (pin "MCU_PERMIT" input (at 195.58 332.74 180) (effects (font (size 1 1)) (justify left))) (pin "GLOW_CMD" input (at 195.58 347.98 180) (effects (font (size 1 1)) (justify left))) (pin "FUEL_CMD" input (at 195.58 355.6 180) (effects (font (size 1 1)) (justify left))) (pin "K_GLOW_COIL_LOW" output (at 381.0 287.02 0) (effects (font (size 1 1)) (justify right))) (pin "K_CLUTCH_RUN_COIL_LOW" output (at 381.0 294.64 0) (effects (font (size 1 1)) (justify right))) (pin "K_CLUTCH_SAFE_COIL_LOW" output (at 381.0 302.26 0) (effects (font (size 1 1)) (justify right))))
 (wire (pts (xy 180.34 76.2) (xy 175.26 76.2)) (stroke (width 0) (type default)))
 (label "P24_PRESENT" (at 175.26 76.2 0) (effects (font (size 1 1)) (justify right bottom)))
 (no_connect (at 251.46 101.6))
+(no_connect
+	(at 180.34 73.66)
+)
+(no_connect
+	(at 180.34 88.9)
+)
+(no_connect
+	(at 251.46 78.74)
+)
 )

Commit message: hardware: remove external EN_CHIP_PU path
Connections:
- net EN_CHIP_PU: no longer names the net of J1.3 (Pin_3)
- no-connect marks 23 -> 24
Other:
- note added: "Manual RESET removed: no J24, external reset header, jumper or replacement button. Automatic safety remains: watchdog, latch and CLEAR_N conditions are preserved. U6.4 is fixed HIGH by +3V3; valid arming requires a new ARM_PULSE from ESP32. Legacy external EN_CHIP_PU path removed; J1.3 is intentionally NC. DevKit internal EN/button/USB auto-reset remain; firmware synchronization is pending."
- note removed: "Manual RESET removed: no J24, external reset header, jumper or replacement button. Automatic safety remains: watchdog, latch and CLEAR_N conditions are preserved. U6.4 is fixed HIGH by +3V3; valid arming requires a new ARM_PULSE from ESP32. EN_CHIP_PU remains at J1.3 for DevKit/USB service; firmware synchronization is pending."
Changed lines of the file:
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@@
-(wire
-	(pts
-		(xy 180.34 68.58) (xy 177.8 68.58)
-	)
-	(stroke
-		(width 0)
-		(type default)
-	)
-)
 (wire
 	(pts
@@
 		)
 	)
-(label "EN_CHIP_PU"
-		(at 177.8 68.58 180)
-		(effects
-			(font
-				(size 1.27 1.27)
-			)
-			(justify right bottom)
-		)
-	)
 (label "+3V3"
 		(at 289.56 209.55 270)
@@
 	 (justify left top))
 )
-(text "Manual RESET removed: no J24, external reset header, jumper or replacement button.\nAutomatic safety remains: watchdog, latch and CLEAR_N conditions are preserved.\nU6.4 is fixed HIGH by +3V3; valid arming requires a new ARM_PULSE from ESP32.\nEN_CHIP_PU remains at J1.3 for DevKit/USB service; firmware synchronization is pending."
+(text "Manual RESET removed: no J24, external reset header, jumper or replacement button.\nAutomatic safety remains: watchdog, latch and CLEAR_N conditions are preserved.\nU6.4 is fixed HIGH by +3V3; valid arming requires a new ARM_PULSE from ESP32.\nLegacy external EN_CHIP_PU path removed; J1.3 is intentionally NC.\nDevKit internal EN/button/USB auto-reset remain; firmware synchronization is pending."
 	(at 25.4 375.92 0)
 	(effects
@@
 	(at 251.46 78.74)
 )
-)
+(no_connect
+	(at 180.34 68.58)
+)
+)

Commit message: WIP: connect OCP_OK feedback to GPIO18
Connections:
- net OCP_OK: now reaches J1.11 (Pin_11)
- no-connect marks 24 -> 23
Other:
- sheet MOTOR_PWM_REBUILD_CANDIDATE ports: added OCP_OK; removed none
Changed lines of the file:
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@@
+			)
+		)
+		(pin "OCP_OK" output
+			(at 455.93 48.26 0)
+			(effects
+				(font
+					(size 1.27 1.27)
+				)
+				(justify right)
 			)
 		)
@@
 (sheet (at 195.58 271.78) (size 185.42 91.44) (stroke (width 0.1524) (type solid)) (fill (color 0 0 0 0)) (property "Sheetname" "MinimalSafety" (at 195.58 270.51 0) (effects (font (size 1.27 1.27)) (justify left bottom))) (property "Sheetfile" "MinimalSafety.kicad_sch" (at 195.58 364.49 0) (effects (font (size 1 1)) (justify left top))) (pin "GND" input (at 195.58 287.02 180) (effects (font (size 1 1)) (justify left))) (pin "P24_PROTECTED" input (at 195.58 294.64 180) (effects (font (size 1 1)) (justify left))) (pin "MCU_PERMIT" input (at 195.58 332.74 180) (effects (font (size 1 1)) (justify left))) (pin "GLOW_CMD" input (at 195.58 347.98 180) (effects (font (size 1 1)) (justify left))) (pin "FUEL_CMD" input (at 195.58 355.6 180) (effects (font (size 1 1)) (justify left))) (pin "K_GLOW_COIL_LOW" output (at 381.0 287.02 0) (effects (font (size 1 1)) (justify right))) (pin "K_CLUTCH_RUN_COIL_LOW" output (at 381.0 294.64 0) (effects (font (size 1 1)) (justify right))) (pin "K_CLUTCH_SAFE_COIL_LOW" output (at 381.0 302.26 0) (effects (font (size 1 1)) (justify right))))
 (wire (pts (xy 180.34 76.2) (xy 175.26 76.2)) (stroke (width 0) (type default)))
+(wire
+	(pts
+		(xy 180.34 88.9) (xy 177.8 88.9)
+	)
+	(stroke
+		(width 0)
+		(type default)
+	)
+)
+(wire
+	(pts
+		(xy 455.93 48.26) (xy 461.01 48.26)
+	)
+	(stroke
+		(width 0)
+		(type default)
+	)
+)
 (label "P24_PRESENT" (at 175.26 76.2 0) (effects (font (size 1 1)) (justify right bottom)))
+(label "OCP_OK"
+		(at 177.8 88.9 180)
+		(effects
+			(font
+				(size 1.27 1.27)
+			)
+			(justify right bottom)
+		)
+	)
+(label "OCP_OK"
+		(at 461.01 48.26 0)
+		(effects
+			(font
+				(size 1.27 1.27)
+			)
+			(justify left bottom)
+		)
+	)
 (no_connect (at 251.46 101.6))
 (no_connect
@@
 )
 (no_connect
-	(at 180.34 88.9)
-)
-(no_connect
