File: hardware/kicad/Sirokko26201_control_motor_candidate.kicad_sch (KiCad schematic)
At the start: 48 parts, among them J1 DEVKITC1_J1, J10 TC_K_EXHAUST_T+_T-, J11 TC_K_AIR_T+_T-, J12 ROOM_DS18B20_HARNESS, J13 24V_INPUT_PHOENIX_1756993_WIP, J22 START_STOP B3F-4055 + B32-138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, J23 ENCODER EC11E15244G1 + KNOB 4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, J26 TFT CABLE HARWIN M20-9960845 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, J27 GLOW_OUTPUT_PHOENIX_1756993, J28 CLUTCH_OUTPUT_PHOENIX_1756993, J3 DEVKITC1_J3, K1 DG85BM-5021-76-1024 + DZ85AB-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, K2 DG85BM-5021-76-1024 + DZ85AB-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, K3 DG85BM-5021-76-1024 + DZ85AB-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, Q20 BC847B,215, U10 MAX31856MUD+, U20 SN74LVC1G97DBVR, U9 MAX31856MUD+

Commit message: Publish current HC-160A CAD snapshot
Connections:
- net OCP_OK: no longer names the net of J1.11 (Pin_11)
- no-connect marks 23 -> 24
Other:
- sheet MOTOR_PWM_REBUILD_CANDIDATE renamed MOTOR_EXTERNAL_HC160
- sheet MOTOR_EXTERNAL_HC160: file motor_pwm_REBUILD.kicad_sch -> motor_external_hc160.kicad_sch
- sheet MOTOR_EXTERNAL_HC160 ports: added none; removed +3V3, OCP_OK, P24_PROTECTED
Changed lines of the file:
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@@
-		)
-	)
-(label "P24_PROTECTED"
-		(at 430.53 43.18 0)
-		(effects
-			(font
-				(size 1.27 1.27)
-			)
-			(justify left bottom)
 		)
 	)
 (label "GND"
 		(at 430.53 45.72 0)
-		(effects
-			(font
-				(size 1.27 1.27)
-			)
-			(justify left bottom)
-		)
-	)
-(label "+3V3"
-		(at 430.53 48.26 0)
 		(effects
 			(font
@@
 			(color 0 0 0 0.0000)
 		)
-		(property "Sheetname" "MOTOR_PWM_REBUILD_CANDIDATE"
+		(property "Sheetname" "MOTOR_EXTERNAL_HC160"
 			(at 430.53 39.9284 0)
 			(effects
@@
 			)
 		)
-		(property "Sheetfile" "motor_pwm_REBUILD.kicad_sch"
+		(property "Sheetfile" "motor_external_hc160.kicad_sch"
 			(at 430.53 51.3846 0)
 			(effects
@@
 				)
 				(justify left top)
-			)
-		)
-		(pin "P24_PROTECTED" input
-			(at 430.53 43.18 180)
-			(effects
-				(font
-					(size 1.27 1.27)
-				)
-				(justify left)
 			)
 		)
@@
 			)
 		)
-		(pin "+3V3" input
-			(at 430.53 48.26 180)
-			(effects
-				(font
-					(size 1.27 1.27)
-				)
-				(justify left)
-			)
-		)
 		(pin "SPEED_CMD" input
 			(at 455.93 43.18 0)
@@
 		(pin "FAN_REQUEST" input
 			(at 455.93 45.72 0)
-			(effects
-				(font
-					(size 1.27 1.27)
-				)
-				(justify right)
-			)
-		)
-		(pin "OCP_OK" output
-			(at 455.93 48.26 0)
 			(effects
 				(font
@@
 (sheet (at 195.58 271.78) (size 185.42 91.44) (stroke (width 0.1524) (type solid)) (fill (color 0 0 0 0)) (property "Sheetname" "MinimalSafety" (at 195.58 270.51 0) (effects (font (size 1.27 1.27)) (justify left bottom))) (property "Sheetfile" "MinimalSafety.kicad_sch" (at 195.58 364.49 0) (effects (font (size 1 1)) (justify left top))) (pin "GND" input (at 195.58 287.02 180) (effects (font (size 1 1)) (justify left))) (pin "P24_PROTECTED" input (at 195.58 294.64 180) (effects (font (size 1 1)) (justify left))) (pin "MCU_PERMIT" input (at 195.58 332.74 180) (effects (font (size 1 1)) (justify left))) (pin "GLOW_CMD" input (at 195.58 347.98 180) (effects (font (size 1 1)) (justify left))) (pin "FUEL_CMD" input (at 195.58 355.6 180) (effects (font (size 1 1)) (justify left))) (pin "K_GLOW_COIL_LOW" output (at 381.0 287.02 0) (effects (font (size 1 1)) (justify right))) (pin "K_CLUTCH_RUN_COIL_LOW" output (at 381.0 294.64 0) (effects (font (size 1 1)) (justify right))) (pin "K_CLUTCH_SAFE_COIL_LOW" output (at 381.0 302.26 0) (effects (font (size 1 1)) (justify right))))
 (wire (pts (xy 180.34 76.2) (xy 175.26 76.2)) (stroke (width 0) (type default)))
-(wire
-	(pts
-		(xy 180.34 88.9) (xy 177.8 88.9)
-	)
-	(stroke
-		(width 0)
-		(type default)
-	)
-)
-(wire
-	(pts
-		(xy 455.93 48.26) (xy 461.01 48.26)
-	)
-	(stroke
-		(width 0)
-		(type default)
-	)
-)
 (label "P24_PRESENT" (at 175.26 76.2 0) (effects (font (size 1 1)) (justify right bottom)))
-(label "OCP_OK"
-		(at 177.8 88.9 180)
-		(effects
-			(font
-				(size 1.27 1.27)
-			)
-			(justify right bottom)
-		)
-	)
-(label "OCP_OK"
-		(at 461.01 48.26 0)
-		(effects
-			(font
-				(size 1.27 1.27)
-			)
-			(justify left bottom)
-		)
-	)
 (no_connect (at 251.46 101.6))
 (no_connect
@@
 	(at 180.34 68.58)
 )
-)
+(no_connect
+	(at 180.34 88.9)
+)
+)

Commit message: Publish DFR0650 schematic WIP
Parts:
- removed DS1: Waveshare 18366 / 2.4inch LCD Module, Sirokko_Mechanical:Waveshare_18366_Module_Bside_Envelope_NO_CY, symbol Sirokko_Mechanical:Waveshare_18366_Module
- removed J26: TFT CABLE HARWIN M20-9960845 RA THT, Sirokko_Connectors:Harwin_M20_9960845_1x08_P2.54mm_RA_THT_Bside, symbol Connector_Generic:Conn_01x08
- removed R24: 10k TFT_CS_PULLUP, Resistor_SMD:R_0603_1608Metric, symbol Device:R
- added C307: 100nF, Capacitor_SMD:C_0603_1608Metric, symbol Device:C
- added DS1: DFRobot DFR0650 / I2C 0x3C / 3.3V, Connector_PinSocket_2.54mm:PinSocket_1x06_P2.54mm_Vertical, symbol Connector_Generic:Conn_01x06
Connections:
- net +3V3: now also C307.1, DS1.1 (Pin_1)
- net GND: now also C307.2, DS1.2 (Pin_2)
- net TFT_CS renamed OLED_SCL
- net OLED_SCL: now also DS1.3 (Pin_3)
- net TFT_DC renamed OLED_SDA
- net OLED_SDA: now also DS1.4 (Pin_4)
- no-connect marks 24 -> 26
Other:
- removed sheet TFT_POWER_3V3_DRAFT
- removed sheet TFT_RESET_LOCAL_DRAFT
- removed sheet TFT_SPI_ISOLATION_DRAFT
- note added: "DEFINED INPUTS / OUTPUTS R1: room-sensor pull-up; R2/R3: thermocouple CS pull-ups. R7/R8: fan/PWM pulldowns. Safety pull resistors are inside MinimalSafety. GPIO21 MCU_PERMIT and GPIO41 ARM_PULSE are outputs; GPIO6 P24_PRESENT is INPUT ONLY. GPIO8 = OLED_SDA; GPIO47 = OLED_SCL; GPIO48 remains for the DevKit RGB LED. No RGB jumper removal. GPIO42 / former SW_TRIP is unconnected. New firmware only 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"
- note removed: "DEFINED INPUTS / OUTPUTS R1: room-sensor pull-up; R2/R3: thermocouple CS pull-ups. R7/R8: fan/PWM pulldowns. Safety pull resistors are inside MinimalSafety. GPIO21 MCU_PERMIT and GPIO41 ARM_PULSE are outputs; GPIO6 P24_PRESENT is INPUT ONLY. GPIO8 = TFT_DC; GPIO48 remains for the DevKit RGB LED. No RGB jumper removal. GPIO42 / former SW_TRIP is unconnected. New firmware only after PCB completion."

Commit message: Publish low-cost OLED schematic WIP
Parts:
- removed DS1: DFRobot DFR0650 / I2C 0x3C / 3.3V, Connector_PinSocket_2.54mm:PinSocket_1x06_P2.54mm_Vertical, symbol Connector_Generic:Conn_01x06
- added DS1: OLED I2C 128x64 / ChipDip 9001709304, Connector_PinSocket_2.54mm:PinSocket_1x04_P2.54mm_Vertical, symbol Connector_Generic:Conn_01x04
Connections:
- net +3V3: now also DS1.2 (Pin_2)
- net GND: now also DS1.1 (Pin_1)
- net OLED_SCL: now also DS1.3 (Pin_3)
- net OLED_SDA: now also DS1.4 (Pin_4)
- no-connect marks 26 -> 24
Changed lines of the file:
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@@
 )
 (symbol
-	(lib_name "Connector_Generic:Conn_01x06")
-	(lib_id "Connector_Generic:Conn_01x06")
-	(at 340.36 205.74 0)
+	(lib_name "Device:C")
+	(lib_id "Device:C")
+	(at 309.88 205.74 0)
 	(unit 1)
 	(exclude_from_sim no)
@@
 	(on_board yes)
 	(dnp no)
-	(property "Reference" "DS1"
-		(at 345.44 198.12 0)
+	(property "Reference" "C307"
+		(at 303.53 205.74 0)
 		(effects
 			(font
@@
 		)
 	)
-	(property "Value" "DFRobot DFR0650 / I2C 0x3C / 3.3V"
-		(at 350.52 219.71 0)
+	(property "Value" "100nF"
+		(at 309.88 213.36 0)
 		(effects
 			(font
@@
 		)
 	)
-	(property "Footprint" "Connector_PinSocket_2.54mm:PinSocket_1x06_P2.54mm_Vertical"
-		(at 340.36 205.74 0)
+	(property "Footprint" "Capacitor_SMD:C_0603_1608Metric"
+		(at 309.88 205.74 0)
 		(effects
 			(font
@@
 		)
 	)
-	(property "Datasheet" "https://wiki.dfrobot.com/Monochrome_0.96_128x64_IIC_SPI_OLED_Display_SKU_DFR0650"
-		(at 340.36 205.74 0)
+	(property "Datasheet" "~"
+		(at 309.88 205.74 0)
 		(effects
 			(font
@@
 		)
 	)
+	(property "MPN" "GRM188R71E104KA01D"
+	(id 0)
+	(at 309.88 205.74 0)
+	(effects
+		(font
+			(size 1.27 1.27)
+		)
+		(hide yes)
+	)
+)
 	(pin "1"
 )
 	(pin "2"
 )
-	(pin "3"
-)
-	(pin "4"
-)
-	(pin "5"
-)
-	(pin "6"
-)
 	(instances
 		(project "Sirokko26201_control_motor_candidate"
 			(path "/d7270d3f-3491-4796-ae0a-c336632ea3f7"
-				(reference "DS1")
+				(reference "C307")
 				(unit 1)
 			)
@@
 )
 (symbol
-	(lib_name "Device:C")
-	(lib_id "Device:C")
-	(at 309.88 205.74 0)
+	(lib_name "Connector_Generic:Conn_01x04")
+	(lib_id "Connector_Generic:Conn_01x04")
+	(at 340.36 203.2 0)
 	(unit 1)
 	(exclude_from_sim no)
@@
 	(on_board yes)
 	(dnp no)
-	(property "Reference" "C307"
-		(at 303.53 205.74 0)
+	(property "Reference" "DS1"
+		(at 345.44 198.12 0)
 		(effects
 			(font
@@
 		)
 	)
-	(property "Value" "100nF"
-		(at 309.88 213.36 0)
+	(property "Value" "OLED I2C 128x64 / ChipDip 9001709304"
+		(at 353.06 215.9 0)
 		(effects
 			(font
@@
 		)
 	)
-	(property "Footprint" "Capacitor_SMD:C_0603_1608Metric"
-		(at 309.88 205.74 0)
+	(property "Footprint" "Connector_PinSocket_2.54mm:PinSocket_1x04_P2.54mm_Vertical"
+		(at 340.36 203.2 0)
 		(effects
 			(font
@@
 		)
 	)
-	(property "Datasheet" "~"
-		(at 309.88 205.74 0)
+	(property "Datasheet" "https://www.chipdip.ru/product/oled-0-96-i2c-belyy-9001709304"
+		(at 340.36 203.2 0)
 		(effects
 			(font
@@
 		)
 	)
-	(property "MPN" "GRM188R71E104KA01D"
-	(id 0)
-	(at 309.88 205.74 0)
-	(effects
-		(font
-			(size 1.27 1.27)
-		)
-		(hide yes)
-	)
-)
 	(pin "1"
 )
 	(pin "2"
 )
+	(pin "3"
+)
+	(pin "4"
+)
 	(instances
 		(project "Sirokko26201_control_motor_candidate"
 			(path "/d7270d3f-3491-4796-ae0a-c336632ea3f7"
-				(reference "C307")
+				(reference "DS1")
 				(unit 1)
 			)
@@
 			(footprint "Capacitor_SMD:C_0805_2012Metric")
 		)
-		(path "/d7270d3f-3491-4796-ae0a-c336632ea3f7/0afd5f5d-db2f-4154-824e-a82de3e3fe5c"
-			(reference "DS1")
-			(unit 1)
-			(value "DFRobot DFR0650 / I2C 0x3C / 3.3V")
-			(footprint "Connector_PinSocket_2.54mm:PinSocket_1x06_P2.54mm_Vertical")
-		)
 		(path "/d7270d3f-3491-4796-ae0a-c336632ea3f7/760ae074-f46f-41f2-ad7d-e66de5977df3"
 			(reference "C307")
@@
 			(footprint "Capacitor_SMD:C_0603_1608Metric")
 		)
+		(path "/d7270d3f-3491-4796-ae0a-c336632ea3f7/dbea4d63-5a50-41de-a6ff-95908133554a"
+			(reference "DS1")
+			(unit 1)
+			(value "OLED I2C 128x64 / ChipDip 9001709304")
+			(footprint "Connector_PinSocket_2.54mm:PinSocket_1x04_P2.54mm_Vertical")
+		)
 )
 (wire
@@
 	(at 180.34 88.9)
 )
-(label "+3V3" (at 320.04 200.66 0) (effects (font (size 1.27 1.27)) (justify left bottom)))
-(label "GND" (at 320.04 203.2 0) (effects (font (size 1.27 1.27)) (justify left bottom)))
+(label "GND" (at 320.04 200.66 0) (effects (font (size 1.27 1.27)) (justify left bottom)))
+(label "+3V3" (at 320.04 203.2 0) (effects (font (size 1.27 1.27)) (justify left bottom)))
 (label "OLED_SCL" (at 320.04 205.74 0) (effects (font (size 1.27 1.27)) (justify left bottom)))
 (label "OLED_SDA" (at 320.04 208.28 0) (effects (font (size 1.27 1.27)) (justify left bottom)))
@@
 		)
 	)
-(no_connect (at 335.28 210.82))
-(no_connect (at 335.28 213.36))
 (wire (pts (xy 320.04 200.66) (xy 335.28 200.66)) (stroke (width 0) (type default)))
 (wire (pts (xy 320.04 203.2) (xy 335.28 203.2)) (stroke (width 0) (type default)))

Commit message: Publish remote-only WIP schematic snapshot
Parts:
- removed C19: 10n ENC_A_FILTER, Capacitor_SMD:C_0603_1608Metric_Pad1.08x0.95mm_HandSolder, symbol Device:C
- removed C20: 10n ENC_B_FILTER, Capacitor_SMD:C_0603_1608Metric_Pad1.08x0.95mm_HandSolder, symbol Device:C
- removed C307: 100nF, Capacitor_SMD:C_0603_1608Metric, symbol Device:C
- removed C75: 10n, Capacitor_SMD:C_0603_1608Metric_Pad1.08x0.95mm_HandSolder, symbol Device:C
- removed DS1: OLED I2C 128x64 / ChipDip 9001709304, Connector_PinSocket_2.54mm:PinSocket_1x04_P2.54mm_Vertical, symbol Connector_Generic:Conn_01x04
- removed J22: START_STOP B3F-4055 + B32-1380 RED, Button_Switch_THT:SW_SPST_Omron_B3F-40xx, symbol Switch:SW_Push
- removed J23: ENCODER EC11E15244G1 + KNOB 41001-1, Sirokko_Panel:RotaryEncoder_Alps_EC11E15244G1_Knob41001_3D_ENVELOPE, symbol Connector_Generic:Conn_01x05
- removed R14: 10k, Resistor_THT:R_Axial_DIN0207_L6.3mm_D2.5mm_P10.16mm_Horizontal, symbol Device:R
- removed R16: 2.2k ENC_A_PULLUP, Resistor_THT:R_Axial_DIN0207_L6.3mm_D2.5mm_P10.16mm_Horizontal, symbol Device:R
- removed R17: 2.2k ENC_B_PULLUP, Resistor_THT:R_Axial_DIN0207_L6.3mm_D2.5mm_P10.16mm_Horizontal, symbol Device:R
- removed R85: 2.2k, Resistor_SMD:R_0603_1608Metric_Pad0.98x0.95mm_HandSolder, symbol Device:R
Connections:
- net ENC_A: no longer names the net of J3.9 (Pin_9)
- net ENC_B: no longer names the net of J3.8 (Pin_8)
- net ENC_SW: no longer names the net of J3.10 (Pin_10)
- net OLED_SCL: no longer names the net of J3.17 (Pin_17)
- net OLED_SDA: no longer names the net of J1.12 (Pin_12)
- net START_REQUEST: no longer names the net of J1.7 (Pin_7)
- no-connect marks 24 -> 30
Other:
- note added: "DEFINED INPUTS / OUTPUTS - REMOTE CONTROL ONLY R1: room-sensor pull-up; R2/R3: thermocouple CS pull-ups. R7/R8: fan/PWM pulldowns. Relay driver resistors remain inside MinimalSafety. No display, encoder or Start/Stop button. Their six former DevKit pins are NC. Remote commands are handled by ESP32; no new control connector is added. Firmware and remote link-loss behavior remain to be implemented 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"
- note added: "NO LOCAL USER CONTROLS / DRAFT No display, Start/Stop, encoder or separate RESET on this carrier. No replacement UI header, jumper or local arming control. Old external watchdog/latch circuitry is not restored. DevKit built-in EN/BOOT and USB programming circuitry are unchanged. No automatic heater restart after reset or a restored remote link."
- note removed: "DEFINED INPUTS / OUTPUTS R1: room-sensor pull-up; R2/R3: thermocouple CS pull-ups. R7/R8: fan/PWM pulldowns. Safety pull resistors are inside MinimalSafety. GPIO21 MCU_PERMIT and GPIO41 ARM_PULSE are outputs; GPIO6 P24_PRESENT is INPUT ONLY. GPIO8 = OLED_SDA; GPIO47 = OLED_SCL; GPIO48 remains for the DevKit RGB LED. No RGB jumper removal. GPIO42 / former SW_TRIP is unconnected. New firmware only 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"
- note removed: "Manual RESET removed: no J24, external reset header, jumper or replacement button. Automatic safety remains: watchdog, latch and CLEAR_N conditions are preserved. U6.4 is fixed HIGH by +3V3; valid arming requires a new ARM_PULSE from ESP32. Legacy external EN_CHIP_PU path removed; J1.3 is intentionally NC. DevKit internal EN/button/USB auto-reset remain; firmware synchronization is pending."
