File: hardware/kicad/Sirokko_Input_Protection_WIP.kicad_sch (KiCad schematic)
At the start: 17 parts, among them Q1 IPB017N10N5LFATMA1 WIP, Q2 IPB017N10N5LFATMA1 WIP, Q3 IPB017N10N5LFATMA1 WIP, Q4 IPB017N10N5LFATMA1 WIP, U13 LM74800QDRRRQ1 WIP_NOT_TRANSI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

Commit message: Publish DRC-complete CAD draft
Parts:
- C25: symbol Device:C -> Sirokko_Interface:C_Sirokko
- F1: symbol Device:Fuse -> Sirokko_Interface:Fuse_Sirokko
Changed lines of the file:
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@@
 	)
 	(symbol
-		(lib_id "Device:C")
+		(lib_id "Sirokko_Interface:C_Sirokko")
 		(at 149.86 105.41 0)
 		(unit 1)
@@
 	)
 	(symbol
-		(lib_id "Device:Fuse")
+		(lib_id "Sirokko_Interface:Fuse_Sirokko")
 		(at 49.53 49.53 0)
 		(unit 1)
