File: hardware/kicad/motor_external_hc160.kicad_sch (KiCad schematic)
At the start: 1 part, among them J29 HC160_A1_A2_PA_G_CONTROL_ONLY

Commit message: Publish J29 metadata and draft interface BOM
Parts:
- J29: MPN (none) -> 1715747; Manufacturer (none) -> Phoenix Contact
Changed lines of the file:
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@@
 		)
 	)
-	(property "Datasheet" "~"
+	(property "Datasheet" "https://www.phoenixcontact.com/en-pc/products/pcb-terminal-block-mkds-15-4-508-1715747"
 		(at 101.6 76.2 0)
 		(effects
@@
 		)
 	)
+	(property "MPN" "1715747"
+	(id 0)
+	(at 101.6 76.2 0)
+	(effects
+		(font
+			(size 1.27 1.27)
+		)
+		(hide yes)
+	)
+)
+	(property "Manufacturer" "Phoenix Contact"
+	(id 1)
+	(at 101.6 76.2 0)
+	(effects
+		(font
+			(size 1.27 1.27)
+		)
+		(hide yes)
+	)
+)
 	(pin "1"
 )

Commit message: Publish DRC-complete CAD draft
Parts:
- J29: symbol Connector_Generic:Conn_01x04 -> Sirokko_Interface:Conn_01x04_Sirokko
Changed lines of the file:
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@@
 	(paper "A4")
 	(symbol
-	(lib_name "Connector_Generic:Conn_01x04")
-	(lib_id "Connector_Generic:Conn_01x04")
+	(lib_name "Sirokko_Interface:Conn_01x04_Sirokko")
+	(lib_id "Sirokko_Interface:Conn_01x04_Sirokko")
 	(at 101.6 76.2 0)
 	(unit 1)
