File: hardware/candidates/unified_motor_spi_working/Sirokko26201_control_motor_candidate.kicad_pcb (KiCad board)
At the start: 2 copper layers, 180 x 170 mm, 112 parts, among them J1 DEVKITC1_J1, J10 TC_K_EXHAUST_T+_T-, J102 MOTOR_24V_HIGH_SPEED; 125W_HE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, J11 TC_K_AIR_T+_T-, J12 ROOM_DS18B20_HARNESS, J13 24V_LOGIC_INPUT_ONLY__DRAFT_N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, J22 PANEL_DRY_CONTACTS_3V3, J23 LOCAL_BUTTONS_3V3__SET_UP_DOW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, J24 RESET_HW_SPDT_BBM_3V3, J25 THERMAL_AND_HW_ENABLE_3V3_ONLY, J26 TFT_GMT020-02-7P_ST7789V_7P_S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, J3 DEVKITC1_J3, Q101 IRFB4110PBF (100V; RDS(on) @ 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, U1 TPS3431SDRBR, U10 MAX31856MUD+, U101 LM5013DDAR, U2 SN74HCS74D, U3 SN74HCS14D, U4 SN74HCS30D, U5 SN74HCS30D, U6 SN74HCS11D, U7 TPS3839G33DBZR, U8 SN74LVC1G14DBVR, U9 MAX31856MUD+, U9001 LTC7001IMSE#PBF; MSOP-10 EP, U9002 INA240A1ID, U9003 LMV331M5X/NOPB, U9004 SN74LVC1G32DBVR, U9005 SN74LVC1G08DBVR, U9006 SN74LVC1G08DBVR, U9007 LM317HVT/NOPB TO-220; TJ 0…12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

Commit message: hardware: WIP Kelvin routes R9001/INA240 340/78, DRC 180
Parts:
- moved C9004 67.0 mm to (165.8, 156.6)
- moved U9002 10.3 mm to (160.0, 156.0)
Routing:
- net /GND: track 682.3 -> 695.2 mm
- net /MOTOR_PWM_REBUILD_CANDIDATE/MOTOR_POS: track 0.00 -> 7.60 mm
- net /MOTOR_PWM_REBUILD_CANDIDATE/SW_SHUNT_HI: track 0.00 -> 7.60 mm
- net /+3V3: track 457.2 -> 459.7 mm
Changed lines of the file:
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@@
 	(footprint "Package_SO:SOIC-8_3.9x4.9mm_P1.27mm"
 		(layer "F.Cu")
-		(at 155 165)
+		(at 160 156)
 		(descr "SOIC, 8 Pin (JEDEC MS-012AA, https://www.analog.com/media/en/package-pcb-resources/package/pkg_pdf/soic_narrow-r/r_8.pdf)")
 		(tags "SOIC SO")
 		(property "Reference" "U9002"
-			(at 0 -3.4 0)
+			(at 0 4.5 0)
 			(layer "F.SilkS")
 			(effects
@@
 		(tags "Vishay WSLP2726 2mOhm Kelvin current-sense 5W")
 		(property "Reference" "R9001"
-			(at 0 -4.55 270)
+			(at -5 0 0)
 			(layer "F.SilkS")
 			(effects
@@
 	(footprint "Capacitor_SMD:C_0603_1608Metric"
 		(layer "F.Cu")
-		(at 100 169)
+		(at 165.8 156.635)
 		(descr "Capacitor SMD 0603 (1608 Metric), square (rectangular) end terminal, IPC-7351 nominal, (Body size source: IPC-SM-782 page 76, https://www.pcb-3d.com/wordpress/wp-content/uploads/ipc-sm-782a_amendment_1_and_2.pdf)")
 		(tags "capacitor")
 		(property "Reference" "C9004"
-			(at 0 -1.43 0)
+			(at 0.2 2.165 0)
 			(layer "F.SilkS")
 			(effects
@@
 	)
 	(segment
+		(start 162.475 156.635)
+		(end 165.025 156.635)
+		(width 0.4)
+		(layer "F.Cu")
+		(net "/+3V3")
+	)
+	(segment
 		(start 36 61.19)
 		(end 36 65)
@@
 	)
 	(segment
+		(start 166.575 156.635)
+		(end 166.575 155.365)
+		(width 0.4)
+		(layer "F.Cu")
+		(net "/GND")
+	)
+	(segment
 		(start 38.975 61.19)
 		(end 39.7 60.465)
@@
 	)
 	(segment
+		(start 157.525 156.635)
+		(end 157.525 157.905)
+		(width 0.4)
+		(layer "F.Cu")
+		(net "/GND")
+	)
+	(segment
 		(start 78 64)
 		(end 78 79.8)
@@
 	)
 	(segment
+		(start 166.575 155.365)
+		(end 162.475 155.365)
+		(width 0.4)
+		(layer "F.Cu")
+		(net "/GND")
+	)
+	(segment
 		(start 143.04 45.72)
 		(end 143.04 43.525)
@@
 	)
 	(segment
+		(start 157.525 155.365)
+		(end 162.475 155.365)
+		(width 0.4)
+		(layer "F.Cu")
+		(net "/GND")
+	)
+	(segment
 		(start 71 79.8)
 		(end 71 75)
@@
 	)
 	(segment
+		(start 157.525 155.365)
+		(end 157.525 156.635)
+		(width 0.4)
+		(layer "F.Cu")
+		(net "/GND")
+	)
+	(segment
 		(start 29.525 68.81)
 		(end 28.2 68.81)
@@
 	)
 	(segment
+		(start 157.525 153.525)
+		(end 157.525 154.095)
+		(width 0.25)
+		(layer "F.Cu")
+		(net "/MOTOR_PWM_REBUILD_CANDIDATE/MOTOR_POS")
+	)
+	(segment
+		(start 157.535 148.295)
+		(end 159.7 150.46)
+		(width 0.25)
+		(layer "F.Cu")
+		(net "/MOTOR_PWM_REBUILD_CANDIDATE/MOTOR_POS")
+	)
+	(segment
+		(start 159.7 151.35)
+		(end 157.525 153.525)
+		(width 0.25)
+		(layer "F.Cu")
+		(net "/MOTOR_PWM_REBUILD_CANDIDATE/MOTOR_POS")
+	)
+	(segment
+		(start 159.7 150.46)
+		(end 159.7 151.35)
+		(width 0.25)
+		(layer "F.Cu")
+		(net "/MOTOR_PWM_REBUILD_CANDIDATE/MOTOR_POS")
+	)
+	(segment
+		(start 162.475 153.525)
+		(end 162.475 154.095)
+		(width 0.25)
+		(layer "F.Cu")
+		(net "/MOTOR_PWM_REBUILD_CANDIDATE/SW_SHUNT_HI")
+	)
+	(segment
+		(start 160.3 151.35)
+		(end 162.475 153.525)
+		(width 0.25)
+		(layer "F.Cu")
+		(net "/MOTOR_PWM_REBUILD_CANDIDATE/SW_SHUNT_HI")
+	)
+	(segment
+		(start 160.3 150.46)
+		(end 160.3 151.35)
+		(width 0.25)
+		(layer "F.Cu")
+		(net "/MOTOR_PWM_REBUILD_CANDIDATE/SW_SHUNT_HI")
+	)
+	(segment
+		(start 162.465 148.295)
+		(end 160.3 150.46)
+		(width 0.25)
+		(layer "F.Cu")
+		(net "/MOTOR_PWM_REBUILD_CANDIDATE/SW_SHUNT_HI")
+	)
+	(segment
 		(start 24 29.7)
 		(end 24 31.5)
@@
 			)
 		)
+	)
+	(zone
+		(layer "F.Cu")
+		(name "R9001_KELVIN_NO_ZONE_COPPER")
+		(hatch edge 0.5)
+		(connect_pads
+			(clearance 0)
+		)
+		(min_thickness 0.25)
+		(keepout
+			(tracks allowed)
+			(vias allowed)
+			(pads allowed)
+			(copperpour not_allowed)
+			(footprints allowed)
+		)
+		(placement
+			(enabled no)
+			(sheetname "")
+		)
+		(fill
+			(thermal_gap 0.5)
+			(thermal_bridge_width 0.5)
+			(island_removal_mode 0)
+		)
+		(polygon
+			(pts
+				(xy 155.9 147.6) (xy 164.1 147.6) (xy 164.1 154.6) (xy 155.9 154.6)
+			)
+		)
