File: hardware/candidates/unified_motor_spi_working/Sirokko26201_control_motor_candidate.kicad_pcb (KiCad board)
At the start: 2 copper layers, 180 x 170 mm, 112 parts, among them J1 DEVKITC1_J1, J10 TC_K_EXHAUST_T+_T-, J102 MOTOR_24V_HIGH_SPEED; 125W_HE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, J11 TC_K_AIR_T+_T-, J12 ROOM_DS18B20_HARNESS, J13 24V_LOGIC_INPUT_ONLY__DRAFT_N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, J22 PANEL_DRY_CONTACTS_3V3, J23 LOCAL_BUTTONS_3V3__SET_UP_DOW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, J24 RESET_HW_SPDT_BBM_3V3, J25 THERMAL_AND_HW_ENABLE_3V3_ONLY, J26 TFT_GMT020-02-7P_ST7789V_7P_S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, J3 DEVKITC1_J3, Q101 IRFB4110PBF (100V; RDS(on) @ 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, U1 TPS3431SDRBR, U10 MAX31856MUD+, U101 LM5013DDAR, U2 SN74HCS74D, U3 SN74HCS14D, U4 SN74HCS30D, U5 SN74HCS30D, U6 SN74HCS11D, U7 TPS3839G33DBZR, U8 SN74LVC1G14DBVR, U9 MAX31856MUD+, U9001 LTC7001IMSE#PBF; MSOP-10 EP, U9002 INA240A1ID, U9003 LMV331M5X/NOPB, U9004 SN74LVC1G32DBVR, U9005 SN74LVC1G08DBVR, U9006 SN74LVC1G08DBVR, U9007 LM317HVT/NOPB TO-220; TJ 0…12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

Commit message: hardware: WIP OCP TLV9020 and INA240 routing 375/80, DRC 167
Parts:
- U9003: value LMV331M5X/NOPB -> TLV9020DBVR
- moved R9005 63.3 mm to (163.0, 168.0)
- moved R9006 60.3 mm to (167.0, 168.0)
- moved C9005 51.7 mm to (156.5, 164.9), turned to 180 degrees
- moved R9007 41.9 mm to (155.5, 168.0)
- moved R9008 33.6 mm to (151.5, 160.0)
- moved U9003 32.6 mm to (161.0, 164.0), turned to 180 degrees
Routing:
- net /+3V3: track 459.7 -> 494.9 mm, vias 9 -> 11
- net /GND: track 695.2 -> 721.3 mm
- net /MOTOR_PWM_REBUILD_CANDIDATE/OCP_THRESH: track 0.00 -> 18.5 mm
- net /MOTOR_PWM_REBUILD_CANDIDATE/OCP_OK: track 0.00 -> 17.2 mm
- net /MOTOR_PWM_REBUILD_CANDIDATE/ISENSE_OUT: track 0.00 -> 5.28 mm

Commit message: hardware: WIP mounting keepouts and motor logic 405/82, DRC 158
Parts:
- moved H3 48.0 mm to (18.0, 172.0)
- moved H4 48.0 mm to (182.0, 172.0)
- moved R9002 18.2 mm to (127.9, 153.7), turned to 180 degrees
- moved H1 4.47 mm to (18.0, 20.0)
- moved H2 4.47 mm to (182.0, 20.0)
Routing:
- net /MOTOR_PWM_REBUILD_CANDIDATE/FAN_WORK_PWM: track 0.00 -> 39.1 mm
- net /MOTOR_PWM_REBUILD_CANDIDATE/MOTOR_GATE_CMD: track 0.00 -> 39.1 mm, vias 0 -> 2
- net /MOTOR_PWM_REBUILD_CANDIDATE/FAN_REQUEST_OR_EMERG: track 0.00 -> 12.9 mm
- net /MOTOR_PWM_REBUILD_CANDIDATE/OCP_OK: track 17.2 -> 28.7 mm
- net /GND: track 721.3 -> 732.7 mm
