File: hardware/candidates/unified_motor_spi_working/motor_pwm_REBUILD.kicad_sch (KiCad schematic)
At the start: 26 parts, among them J102 MOTOR_24V_HIGH_SPEED; 125W_HE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, Q101 IRFB4110PBF (100V; RDS(on) @ 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, U9001 LTC7001IMSE#PBF; MSOP-10 EP, U9002 INA240A1ID, U9003 LMV331M5X/NOPB, U9004 SN74LVC1G32DBVR, U9005 SN74LVC1G08DBVR, U9006 SN74LVC1G08DBVR, U9007 LM317HVT/NOPB TO-220; TJ 0…12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

Commit message: hardware: WIP OCP TLV9020 and INA240 routing 375/80, DRC 167
Parts:
- U9003: value LMV331M5X/NOPB -> TLV9020DBVR; symbol Comparator:LMV331 -> Sirokko_Power:TLV9020DBVR
Other:
- note added: "CURRENT INTERFACE - DRAFT: 15 A continuous design limit, not measured motor current. Logic design range +3V3=3.135...3.465 V; 3.0...3.6 V is an additional stress calculation. Nominal ideal OCP at 3.3 V: trip 21.081 A, reset 20.471 A. These are NOT qualified limits. See OCP_TLV9020_REVIEW_RU.md and ocp_threshold_model.json for assumptions. Coordinate branch fuse, wiring, connector, MOSFET SOA and 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"
- note added: "LOGIC CONTRACT - DRAFT, not bench qualified. INP = ((FAN_CMD AND PWM_SPEED_CMD) OR FAN_EMERG_3V3) AND OCP_OK. R9002=100k pulls INP LOW when +3V3/gates are off; VIN/VDRV may remain. U9003 TLV9020DBVR: open-drain OUT4; IN+1, IN-3, V-2, V+5. Overcurrent pulls OCP_OK LOW and inhibits both PWM and emergency command. Verify physical shutdown timing and current decay on a safe bench."
- note removed: "CURRENT INTERFACE: design continuous limit 15 A; comparator trip/release corridor 19.11…22.42 A for +3V3=3.135…3.465 V and 1% resistors. This is hardware turn-off, not a current regulator. External branch fuse/wiring/connector must be selected for the 15 A continuous interface; motor L/I/start profile remains a commissioning measurement."
- note removed: "QUALIFIED LOGIC: INP = ((FAN_CMD AND PWM_SPEED_CMD) OR FAN_EMERG_3V3) AND OCP_OK. R9002=100k pulls INP low. Loss of +3V3 drives gates Hi-Z; R9002 forces LTC7001 INP=LOW even with VIN/VDRV alive. OCP_OK is LMV331 open collector: overcurrent pulls LOW and therefore turns OFF both PWM and emergency command."
Changed lines of the file:
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@@
 )
 	(symbol
-	(lib_name "Comparator:LMV331")
-	(lib_id "Comparator:LMV331")
+	(lib_name "Sirokko_Power:TLV9020DBVR")
+	(lib_id "Sirokko_Power:TLV9020DBVR")
 	(at 149.86 119.38 0)
 	(unit 1)
@@
 	(dnp no)
 	(property "Reference" "U9003"
-		(at 149.86 115.57 0)
-		(effects
-			(font
-				(size 1.27 1.27)
-			)
-		)
-	)
-	(property "Value" "LMV331M5X/NOPB"
-		(at 149.86 123.19 0)
+		(at 155 110 0)
+		(effects
+			(font
+				(size 1.27 1.27)
+			)
+		)
+	)
+	(property "Value" "TLV9020DBVR"
+		(at 155 112.5 0)
 		(effects
 			(font
@@
 		)
 	)
-	(property "Datasheet" "~"
+	(property "Datasheet" "https://www.ti.com/lit/ds/symlink/tlv9021.pdf"
 		(at 149.86 119.38 0)
 		(effects
@@
 	)
 )
-	(text "QUALIFIED LOGIC: INP = ((FAN_CMD AND PWM_SPEED_CMD) OR FAN_EMERG_3V3) AND OCP_OK. R9002=100k pulls INP low. Loss of +3V3 drives gates Hi-Z; R9002 forces LTC7001 INP=LOW even with VIN/VDRV alive. OCP_OK is LMV331 open collector: overcurrent pulls LOW and therefore turns OFF both PWM and emergency command."
+	(text "LOGIC CONTRACT - DRAFT, not bench qualified.\nINP = ((FAN_CMD AND PWM_SPEED_CMD) OR FAN_EMERG_3V3) AND OCP_OK.\nR9002=100k pulls INP LOW when +3V3/gates are off; VIN/VDRV may remain.\nU9003 TLV9020DBVR: open-drain OUT4; IN+1, IN-3, V-2, V+5.\nOvercurrent pulls OCP_OK LOW and inhibits both PWM and emergency command.\nVerify physical shutdown timing and current decay on a safe bench."
 	(at 25.4 25.4 0)
 	(effects
@@
 			(size 1.27 1.27)
 		)
-	)
-)
-	(text "CURRENT INTERFACE: design continuous limit 15 A; comparator trip/release corridor 19.11…22.42 A for +3V3=3.135…3.465 V and 1% resistors. This is hardware turn-off, not a current regulator. External branch fuse/wiring/connector must be selected for the 15 A continuous interface; motor L/I/start profile remains a commissioning measurement."
+		(justify left)
+	)
+)
+	(text "CURRENT INTERFACE - DRAFT: 15 A continuous design limit, not measured motor current.\nLogic design range +3V3=3.135...3.465 V; 3.0...3.6 V is an additional stress calculation.\nNominal ideal OCP at 3.3 V: trip 21.081 A, reset 20.471 A. These are NOT qualified limits.\nSee OCP_TLV9020_REVIEW_RU.md and ocp_threshold_model.json for assumptions.\nCoordinate branch fuse, wiring, connector, MOSFET SOA and actual motor startup before release."
 	(at 25.4 38.1 0)
 	(effects
@@
 			(size 1.27 1.27)
 		)
-	)
-)
+		(justify left)
+	)
+)
