File: hardware/candidates/tft_power_tps62162_standalone_DRAFT/tft_power_tps62162_review_DRAFT.kicad_sch (KiCad schematic)
At the start: 8 parts, among them U301 TPS62162DSGR

Commit message: hardware: assign eight TPS62162 draft footprints
Parts:
- C301, C302: footprint (none) -> Sirokko_TFT_Passives:C_Murata_GRM21B_2012_Reflow
- C303: footprint (none) -> Sirokko_TFT_Passives:C_Murata_GRM188_1608_Reflow
- C304: footprint (none) -> Sirokko_TFT_Passives:C_Murata_GRM32E_3225_Reflow
- L301: footprint (none) -> Sirokko_TFT_Passives:L_Wuerth_744025003_2828_Reflow
- R301, R302: footprint (none) -> Sirokko_TFT_Passives:R_Yageo_RC0603_1608_Reflow
- U301: footprint (none) -> Package_SON:Texas_DSG0008A_WSON-8-1EP_2x2mm_P0.5mm_EP0.9x1.6mm_ThermalVias
Changed lines of the file:
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@@
 		)
 	)
-	(property "Footprint" ""
+	(property "Footprint" "Package_SON:Texas_DSG0008A_WSON-8-1EP_2x2mm_P0.5mm_EP0.9x1.6mm_ThermalVias"
 		(at 114.3 76.2 0)
 		(effects
@@
 		)
 	)
-	(property "Footprint" ""
+	(property "Footprint" "Sirokko_TFT_Passives:L_Wuerth_744025003_2828_Reflow"
 		(at 162.56 68.58 0)
 		(effects
@@
 		)
 	)
-	(property "Footprint" ""
+	(property "Footprint" "Sirokko_TFT_Passives:C_Murata_GRM21B_2012_Reflow"
 		(at 45.72 66.04 0)
 		(effects
@@
 		)
 	)
-	(property "Footprint" ""
+	(property "Footprint" "Sirokko_TFT_Passives:C_Murata_GRM21B_2012_Reflow"
 		(at 45.72 91.44 0)
 		(effects
@@
 		)
 	)
-	(property "Footprint" ""
+	(property "Footprint" "Sirokko_TFT_Passives:C_Murata_GRM188_1608_Reflow"
 		(at 45.72 116.84 0)
 		(effects
@@
 		)
 	)
-	(property "Footprint" ""
+	(property "Footprint" "Sirokko_TFT_Passives:C_Murata_GRM32E_3225_Reflow"
 		(at 195.58 96.52 0)
 		(effects
@@
 		)
 	)
-	(property "Footprint" ""
+	(property "Footprint" "Sirokko_TFT_Passives:R_Yageo_RC0603_1608_Reflow"
 		(at 81.28 40.64 0)
 		(effects
@@
 		)
 	)
-	(property "Footprint" ""
+	(property "Footprint" "Sirokko_TFT_Passives:R_Yageo_RC0603_1608_Reflow"
 		(at 162.56 104.14 0)
 		(effects
